File: BPS-Amperes.sch (KiCad schematic (older format))
At the start: 38 parts, among them J1 ShuntConn, J2 LeaderConn, J3 Conn_01x04, U2 RO-123.3S_HP, U3 LTC6820, U4 HX1188FNL, U5 ADS7042xDCU

Commit message: Fixed connection to leader board
Parts:
- gave numbers to parts that had none: 8
Connections:
- wire segments 149 -> 157
Other:
- moved on the sheet: J2
Changed lines of the file:
@@
 L Connector_Generic:Conn_01x04 J2
 U 1 1 5F0D0A13
-P 9950 3950
-F 0 "J2" H 10030 3942 50  0000 L CNN
-F 1 "LeaderConn" H 10030 3851 50  0000 L CNN
-F 2 "Connector_Molex:Molex_Micro-Fit_3.0_43650-0415_1x04_P3.00mm_Vertical" H 9950 3950 50  0001 C CNN
-F 3 "~" H 9950 3950 50  0001 C CNN
-	1    9950 3950
-	1    0    0    -1
+P 9550 4650
+F 0 "J2" H 9630 4642 50  0000 L CNN
+F 1 "LeaderConn" H 9630 4551 50  0000 L CNN
+F 2 "Connector_Molex:Molex_Micro-Fit_3.0_43650-0415_1x04_P3.00mm_Vertical" H 9550 4650 50  0001 C CNN
+F 3 "~" H 9550 4650 50  0001 C CNN
+	1    9550 4650
+	-1   0    0    -1
 $EndComp
 $Comp
@@
 	9500 3900 9500 3950
 Wire Wire Line
-	9500 3950 9750 3950
-Wire Wire Line
 	9150 4100 9500 4100
 Wire Wire Line
 	9500 4100 9500 4050
-Wire Wire Line
-	9500 4050 9750 4050
 NoConn ~ 9150 4000
-Wire Wire Line
-	9750 4150 9600 4150
-Wire Wire Line
-	9600 4150 9600 4200
-Wire Wire Line
-	9750 3850 9600 3850
-Wire Wire Line
-	9600 3850 9600 3800
-$Comp
-L power:+12V #PWR020
-U 1 1 5F14CAA1
-P 9600 3800
-F 0 "#PWR020" H 9600 3650 50  0001 C CNN
-F 1 "+12V" H 9615 3973 50  0000 C CNN
-F 2 "" H 9600 3800 50  0001 C CNN
-F 3 "" H 9600 3800 50  0001 C CNN
-	1    9600 3800
-	1    0    0    -1
-$EndComp
 $Comp
 L Device:C C1
@@
 Wire Wire Line
 	9800 2200 9800 2150
-$Comp
-L power:GNDPWR #PWR021
-U 1 1 5F16DDBE
-P 9600 4200
-F 0 "#PWR021" H 9600 4000 50  0001 C CNN
-F 1 "GNDPWR" H 9604 4046 50  0000 C CNN
-F 2 "" H 9600 4150 50  0001 C CNN
-F 3 "" H 9600 4150 50  0001 C CNN
-	1    9600 4200
-	1    0    0    -1
-$EndComp
 Connection ~ 1950 2000
 Wire Wire Line
@@
 	1    0    0    -1
 $EndComp
-Connection ~ 3800 2300
 $Comp
 L power:+3.3V #PWR015
@@
 	7925 2350 7550 2350
 $Comp
-L utsvt-chips:INA186A3QDBVRQ1 U?
+L utsvt-chips:INA186A3QDBVRQ1 U1
 U 1 1 6158D574
 P 3650 5600
-F 0 "U?" H 3650 5925 50  0000 C CNN
+F 0 "U1" H 3650 5925 50  0000 C CNN
 F 1 "INA186A3IDDFT " H 3650 5834 50  0000 C CNN
 F 2 "" H 3650 5600 50  0001 C CNN
@@
 	3000 5500 3000 5350
 $Comp
-L power:GND #PWR?
+L power:GND #PWR0104
 U 1 1 615BF0B8
 P 3000 5900
-F 0 "#PWR?" H 3000 5650 50  0001 C CNN
+F 0 "#PWR0104" H 3000 5650 50  0001 C CNN
 F 1 "GND" H 3005 5727 50  0000 C CNN
 F 2 "" H 3000 5900 50  0001 C CNN
@@
 	3000 5800 3300 5800
 $Comp
-L Device:C_Small C?
+L Device:C_Small C10
 U 1 1 615C347C
 P 2850 5500
-F 0 "C?" V 2621 5500 50  0000 C CNN
+F 0 "C10" V 2621 5500 50  0000 C CNN
 F 1 "1uF" V 2712 5500 50  0000 C CNN
 F 2 "" H 2850 5500 50  0001 C CNN
@@
 Connection ~ 3000 5500
 $Comp
-L power:GND #PWR?
+L power:GND #PWR0105
 U 1 1 615C83C1
 P 2700 5600
-F 0 "#PWR?" H 2700 5350 50  0001 C CNN
+F 0 "#PWR0105" H 2700 5350 50  0001 C CNN
 F 1 "GND" H 2705 5427 50  0000 C CNN
 F 2 "" H 2700 5600 50  0001 C CNN
@@
 $EndComp
 $Comp
-L power:+3.3V #PWR?
+L power:+3.3V #PWR0111
 U 1 1 615F5252
 P 2850 3300
-F 0 "#PWR?" H 2850 3150 50  0001 C CNN
+F 0 "#PWR0111" H 2850 3150 50  0001 C CNN
 F 1 "+3.3V" H 2865 3473 50  0000 C CNN
 F 2 "" H 2850 3300 50  0001 C CNN
@@
 	2850 3450 3000 3450
 $Comp
-L power:GND #PWR?
+L power:GND #PWR0112
 U 1 1 615FA9A0
 P 2850 3850
-F 0 "#PWR?" H 2850 3600 50  0001 C CNN
+F 0 "#PWR0112" H 2850 3600 50  0001 C CNN
 F 1 "GND" H 2855 3677 50  0000 C CNN
 F 2 "" H 2850 3850 50  0001 C CNN
@@
 	4000 3450 4000 3300
 $Comp
-L power:+1V5 #PWR?
+L power:+1V5 #PWR0113
 U 1 1 6160D6F2
 P 4000 3300
-F 0 "#PWR?" H 4000 3150 50  0001 C CNN
+F 0 "#PWR0113" H 4000 3150 50  0001 C CNN
 F 1 "+1V5" H 4015 3473 50  0000 C CNN
 F 2 "" H 4000 3300 50  0001 C CNN
@@
 $EndComp
 $Comp
-L power:+3V0 #PWR?
+L power:+3V0 #PWR0114
 U 1 1 6160E4A2
 P 4350 3300
-F 0 "#PWR?" H 4350 3150 50  0001 C CNN
+F 0 "#PWR0114" H 4350 3150 50  0001 C CNN
 F 1 "+3V0" H 4365 3473 50  0000 C CNN
 F 2 "" H 4350 3300 50  0001 C CNN
@@
 	5100 5100 5100 5500
 $Comp
-L power:+3V0 #PWR?
+L power:+3V0 #PWR0115
 U 1 1 6161748C
 P 5000 5400
-F 0 "#PWR?" H 5000 5250 50  0001 C CNN
+F 0 "#PWR0115" H 5000 5250 50  0001 C CNN
 F 1 "+3V0" H 4900 5550 50  0000 C CNN
 F 2 "" H 5000 5400 50  0001 C CNN
@@
 $EndComp
 $Comp
-L power:+1V5 #PWR?
+L power:+1V5 #PWR0116
 U 1 1 616203A7
 P 3200 5700
-F 0 "#PWR?" H 3200 5550 50  0001 C CNN
+F 0 "#PWR0116" H 3200 5550 50  0001 C CNN
 F 1 "+1V5" V 3215 5828 50  0000 L CNN
 F 2 "" H 3200 5700 50  0001 C CNN
@@
 	3200 5700 3300 5700
 $Comp
-L power:+3V0 #PWR?
+L power:+3V0 #PWR0117
 U 1 1 61625C0A
 P 3000 5350
-F 0 "#PWR?" H 3000 5200 50  0001 C CNN
+F 0 "#PWR0117" H 3000 5200 50  0001 C CNN
 F 1 "+3V0" H 3000 5500 50  0000 C CNN
 F 2 "" H 3000 5350 50  0001 C CNN
@@
 $EndComp
 $Comp
-L Device:C_Small C?
+L Device:C_Small C7
 U 1 1 61627A94
 P 2450 3600
-F 0 "C?" H 2542 3646 50  0000 L CNN
+F 0 "C7" H 2542 3646 50  0000 L CNN
 F 1 "100nF" H 2542 3555 50  0000 L CNN
 F 2 "" H 2450 3600 50  0001 C CNN
@@
 	2850 3800 2850 3750
 $Comp
-L Device:C_Small C?
+L Device:C_Small C11
 U 1 1 6163F45A
 P 3900 3750
-F 0 "C?" H 3992 3796 50  0000 L CNN
+F 0 "C11" H 3992 3796 50  0000 L CNN
 F 1 "100nF" H 3992 3705 50  0000 L CNN
 F 2 "" H 3900 3750 50  0001 C CNN
@@
 $EndComp
 $Comp
-L Device:C_Small C?
+L Device:C_Small C12
 U 1 1 6163F9FF
 P 4350 3750
-F 0 "C?" H 4442 3796 50  0000 L CNN
+F 0 "C12" H 4442 3796 50  0000 L CNN
 F 1 "100nF" H 4442 3705 50  0000 L CNN
 F 2 "" H 4350 3750 50  0001 C CNN
@@
 $EndComp
 $Comp
-L power:GND #PWR?
+L power:GND #PWR0118
 U 1 1 6163FE48
 P 4150 3950
-F 0 "#PWR?" H 4150 3700 50  0001 C CNN
+F 0 "#PWR0118" H 4150 3700 50  0001 C CNN
 F 1 "GND" H 4250 3800 50  0000 C CNN
 F 2 "" H 4150 3950 50  0001 C CNN
@@
 $EndComp
 $Comp
-L Device:R_Small_US R?
+L Device:R_Small_US R3
 U 1 1 61669A4C
 P 1450 5850
-F 0 "R?" V 1650 5850 50  0000 C CNN
+F 0 "R3" V 1650 5850 50  0000 C CNN
 F 1 "500" V 1550 5850 50  0000 C CNN
 F 2 "" H 1450 5850 50  0001 C CNN
@@
 $EndComp
 $Comp
-L Device:R_Small_US R?
+L Device:R_Small_US R1
 U 1 1 6166A121
 P 1450 5750
-F 0 "R?" V 1250 5750 50  0000 C CNN
+F 0 "R1" V 1250 5750 50  0000 C CNN
 F 1 "500" V 1350 5750 50  0000 C CNN
 F 2 "" H 1450 5750 50  0001 C CNN
@@
 $EndComp
 $Comp
-L Device:C_Small C?
+L Device:C_Small C6
 U 1 1 6166CD6D
 P 1750 5800
-F 0 "C?" H 1842 5846 50  0000 L CNN
+F 0 "C6" H 1842 5846 50  0000 L CNN
 F 1 "22uF" H 1842 5755 50  0000 L CNN
 F 2 "" H 1750 5800 50  0001 C CNN
@@
 Wire Wire Line
 	2150 5700 2450 5700
+$Comp
+L power:+12V #PWR020
+U 1 1 5F14CAA1
+P 9600 3800
+F 0 "#PWR020" H 9600 3650 50  0001 C CNN
+F 1 "+12V" H 9615 3973 50  0000 C CNN
+F 2 "" H 9600 3800 50  0001 C CNN
+F 3 "" H 9600 3800 50  0001 C CNN
+	1    9600 3800
+	1    0    0    -1
+$EndComp
+Wire Wire Line
+	9600 3850 9600 3800
+$Comp
+L power:GNDPWR #PWR021
+U 1 1 5F16DDBE
+P 9600 4200
+F 0 "#PWR021" H 9600 4000 50  0001 C CNN
+F 1 "GNDPWR" H 9604 4046 50  0000 C CNN
+F 2 "" H 9600 4150 50  0001 C CNN
+F 3 "" H 9600 4150 50  0001 C CNN
+	1    9600 4200
+	1    0    0    -1
+$EndComp
+Wire Wire Line
+	9600 4150 9600 4200
+Wire Wire Line
+	9850 4150 9850 4550
+Wire Wire Line
+	9850 4550 9750 4550
+Wire Wire Line
+	9600 4150 9850 4150
+Wire Wire Line
+	9950 4050 9950 4650
+Wire Wire Line
+	9950 4650 9750 4650
+Wire Wire Line
+	9500 4050 9950 4050
+Wire Wire Line
+	10050 3950 10050 4750
+Wire Wire Line
+	10050 4750 9750 4750
+Wire Wire Line
+	9500 3950 10050 3950
+Wire Wire Line
+	10150 3850 10150 4850
+Wire Wire Line
+	10150 4850 9750 4850
+Wire Wire Line
+	9600 3850 10150 3850
 $EndSCHEMATC
