File: BPS-AmperesPCB.kicad_sch (KiCad schematic)
At the start: 0 parts

Commit message: workday 1/4
Parts:
- added C1, C3, C7: C, symbol Device:C
- added C2: 2.2uF, Capacitor_SMD:C_0805_2012Metric, symbol Device:C_Small
- added C4: 1n, symbol Device:C
- added C5: 10u, symbol Device:C
- added C6: 2.2n, Capacitor_SMD:C_0805_2012Metric, symbol Device:C
- added D1: PowerOn, LED_SMD:LED_0805_2012Metric, symbol Device:LED
- added J1: ShuntConn, Connector_PinSocket_2.54mm:PinSocket_1x05_P2.54mm_Vertical, symbol Connector_Generic:Conn_01x05
- added R1, R2, R3, R4: 1.2k, Resistor_SMD:R_0805_2012Metric, symbol Device:R_Small_US
- added R5: 1.5k, Resistor_SMD:R_0805_2012Metric, symbol Device:R
- added U1: PeripheralSOM, UTSVT_Special:PeripheralSOM, symbol utsvt-misc:PeripheralSOM
- added U2: INA229AIDGSR, VSSOP10_DGS_TEX, symbol INA229:INA229AIDGSR
- added U3: AMC1300BDWV, Package_SO:SOIC-8_7.5x5.85mm_P1.27mm, symbol Amplifier_Difference:AMC1300BDWV
- added U4: RO-123.3S_HP, UTSVT_ICs:RI3_DC_Converter, symbol utsvt-power-regulators:RO-123.3S_HP
Connections:
- new net: D1.2 (A), R5.2
- new net: C7.1, R3.1, U2.10 (IN+)
- new net: C7.2, R4.1, U2.9 (IN-)
- new net: J1.2 (Pin_2), R1.2
- new net +12V: C4.1, C5.1, U1.22 (+12V_In), U4.2 (+Vin)
- new net +3V3: C3.1, R5.1, U1.10 (VDDA(3.3V)), U1.2 (+3.3V), U1.9 (+3.3V), U2.6 (VS), U3.8 (V+)
- new net +3V3 High: C1.1, J1.5 (Pin_5), U3.1 (V+), U4.4 (+Vout)
- new net GND: C3.2, D1.1 (K), U1.11 (GND), U1.4 (GND), U2.7 (GND), U3.5 (V-)
- new net GND High: C1.2, C6.2, J1.3 (Pin_3), J1.4 (Pin_4), R2.2, U3.4 (V-), U4.3 (-Vout)
- new net GNDPWR: C4.2, C5.2, C6.1, U1.24 (GNDPWR), U4.1 (-Vin)
- new net INN: C2.2, R2.1, U3.3 (-)
- new net INP: C2.1, R1.1, U3.2 (+)
- new net MISO: U1.15 (SPI1_MISO), U2.4 (MISO)
- new net MOSI: U1.17 (SPI1_MOSI), U2.2 (MOSI)
- new net NSS: U1.19 (SPI1_NSS), U2.1 (CS)
- new net OUTN: R4.2, U3.6 (-)
- new net OUTP: R3.2, U3.7 (+)
- new net SCLK: U1.13 (SPI1_SCK), U2.5 (SCLK)
- no-connect marks 0 -> 1
Other:
- removed sheet INA226
- removed sheet INA293
- note added: "Current Sensor"
- note added: "Peripheral Board"
- note added: "Power"

Commit message: 1/18
Parts:
- added C8, C9: 100uF, symbol Device:C
- C1, C3: value C -> 1uF
- C2: value 2.2uF -> 10nF
- R1, R2: value 1.2k -> 10
Connections:
- net +3V3: now also C8.1
- net GND: now also C8.2
- net GND High: now also C9.2
- net +3V3 BATT: now reaches J1.1 (Pin_1)
- net +3V3 BATT: now also C1.1, U3.1 (V+), U4.4 (+Vout), C9.1
- removed net +3V3 High: C1.1, J1.5 (Pin_5), U3.1 (V+), U4.4 (+Vout)
Other:
- note added: "Isolated Amplifier"
- note removed: "Current Sensor"
- moved on the sheet: C1, C2, C3, J1, R1, R2, U3
