File: hardware/HV_Carrier/Power_Mux.kicad_sch (KiCad schematic)
At the start: 8 parts, among them U10 TPS2117DRLR

Commit message: saving
Parts:
- renumbered R70 to R71, R71 to R72, R72 to R73
Changed lines of the file:
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@@
 		(in_pos_files yes)
 		(dnp no)
-		(property "Reference" "R72"
+		(property "Reference" "R73"
 			(at 78.994 67.564 0)
 			(show_name no)
@@
 			(project "PS-HVCarrier"
 				(path "/2365a867-6254-4a7c-9718-f325e0bbac5c/904fa10a-747c-46cf-90d1-33d76069dc5d/b66ae0b0-03e3-4dd0-8364-435fb922b758"
-					(reference "R72")
+					(reference "R73")
 					(unit 1)
 				)
@@
 		(in_pos_files yes)
 		(dnp no)
-		(property "Reference" "R70"
+		(property "Reference" "R71"
 			(at 35.052 59.944 0)
 			(show_name no)
@@
 			(project "PS-HVCarrier"
 				(path "/2365a867-6254-4a7c-9718-f325e0bbac5c/904fa10a-747c-46cf-90d1-33d76069dc5d/b66ae0b0-03e3-4dd0-8364-435fb922b758"
-					(reference "R70")
+					(reference "R71")
 					(unit 1)
 				)
@@
 		(in_pos_files yes)
 		(dnp no)
-		(property "Reference" "R71"
+		(property "Reference" "R72"
 			(at 35.052 67.564 0)
 			(show_name no)
@@
 			(project "PS-HVCarrier"
 				(path "/2365a867-6254-4a7c-9718-f325e0bbac5c/904fa10a-747c-46cf-90d1-33d76069dc5d/b66ae0b0-03e3-4dd0-8364-435fb922b758"
-					(reference "R71")
-					(unit 1)
-				)
+					(reference "R72")
+					(unit 1)
+				)
