File: hardware/HV_Carrier/PS-HVCarrier.kicad_pcb (KiCad board)
At the start: 2 copper layers, 278 parts, among them IC1 TCAN3413DR, IC2 TCAN3413DR, J1 Shunt Breakout Conn, J10 SSA-2-100A, J2 Hall Breakout Conn, J3 IMD_Conn, J4 Voltage Tap, J5 BPS Conn, J6 SWD_Header, J7 SWD, J8 USB_C_Receptacle_USB2.0_16P, J9 LZSR 80-P, Q1 PSMN012-100YS, Q2 PSMN012-100YS, SW1 Reset, SW2 SW_SPDT, U1 LM74502DDFR, U10 AMC3311QDWERQ1, U11 TPS2117DRLR, U12 TLV9002QDRQ1, U13 TLV9002QDRQ1, U14 LMR51635XDDCR, U2 MCP1826S, U3 CDSOT23-T24CAN, U4 CDSOT23-T24CAN, U5 AMC3311QDWERQ1, U6 STM32G473CETx, U7 TLV9002QDRQ1, U8 AMC3311QDWERQ1, U9 AMC3311QDWERQ1, Y1 Crystal

Commit message: updated layout + hall
Parts:
- removed U14: LMR51635XDDCR, LHRS_ICs:DDC0006A-MFG
- added C90: 100n, Capacitor_SMD:C_0603_1608Metric, F.Cu at (190.8, 46.9)
- added C91: 22u, Capacitor_SMD:C_1210_3225Metric_Pad1.33x2.70mm_HandSolder, F.Cu at (205.5, 57.5)
- added C92: 22u, Capacitor_SMD:C_1210_3225Metric_Pad1.33x2.70mm_HandSolder, F.Cu at (201.2, 57.5)
- added C93: 3.3u, Capacitor_SMD:C_0805_2012Metric_Pad1.18x1.45mm_HandSolder, F.Cu at (197.7, 46.5)
- added H1: MountingHole, MountingHole:MountingHole_3.2mm_M3, F.Cu at (25.5, 153.3)
- added H2: MountingHole, MountingHole:MountingHole_3.2mm_M3, F.Cu at (25.5, 161.2)
- added H3: MountingHole, MountingHole:MountingHole_3.2mm_M3, F.Cu at (25.5, 169.2)
- added H4: MountingHole, MountingHole:MountingHole_3.2mm_M3, F.Cu at (25.5, 177.1)
- added IC3: TCAN3413DR, LHRS_Passives:TCAN3413DR, F.Cu at (122.0, 116.4)
- added J12: Discharge Vin, LHRS_Connectors:Molex_Nano-Fit_105309-xx02_1x02_P2.50mm_Vertical, F.Cu at (47.6, 46.1)
- added J13: Charge Vin, LHRS_Connectors:Molex_Nano-Fit_105309-xx02_1x02_P2.50mm_Vertical, F.Cu at (56.0, 46.1)
- added R85: 10k, Resistor_SMD:R_0603_1608Metric_Pad0.98x0.95mm_HandSolder, F.Cu at (105.6, 47.3)
- added R86: 100k, Resistor_SMD:R_0603_1608Metric, F.Cu at (193.5, 44.3)
- added R87: 19.1k, Resistor_SMD:R_0603_1608Metric, F.Cu at (193.5, 42.5)
- added S1: OS102011MS2QN1, OS102011MS2QN1:OS102011MA1QN1, F.Cu at (56.1, 64.9)
- C10, C14, C9: value 0.1u -> 10u; footprint Capacitor_SMD:C_0603_1608Metric_Pad1.08x0.95mm_HandSolder -> Capacitor_SMD:C_0805_2012Metric_Pad1.18x1.45mm_HandSolder
- C12, C6, C7: value 10u -> 0.1u; footprint Capacitor_SMD:C_0805_2012Metric_Pad1.18x1.45mm_HandSolder -> Capacitor_SMD:C_0603_1608Metric_Pad1.08x0.95mm_HandSolder
- C16: value 100p -> 0.1u
- C17, C50, C84: value 1n -> 0.1u
- C18, C51, C60, C69: value 100n -> 100p
- C19, C52, C61, C70: value 100n -> 1n
- C20, C47, C53, C62, C71: value 1n -> 100n
- C23, C42, C56, C65, C74: value 1u -> 100n
- C24, C57, C66, C75: value 10n -> 1n
- C25: value 26p -> 1u
- C26: value 26p -> 10n
- C27: value 10uF -> 10u; footprint Capacitor_SMD:C_0805_2012Metric -> Capacitor_SMD:C_0805_2012Metric_Pad1.18x1.45mm_HandSolder
- C28, C29: value 0.1uF -> 26p
- C30: value 0.1uF -> 10u; footprint Capacitor_SMD:C_0603_1608Metric_Pad1.08x0.95mm_HandSolder -> Capacitor_SMD:C_0805_2012Metric_Pad1.18x1.45mm_HandSolder
- C33, C35: value 1uF -> 0.1uF
- C36, C38: value 0.1uF -> 1uF
- C39, C41: value 100n -> 0.1uF
- C40: value 10uF -> 0.1uF; footprint Capacitor_SMD:C_0805_2012Metric -> Capacitor_SMD:C_0603_1608Metric_Pad1.08x0.95mm_HandSolder
- C43: value 10n -> 100n
- C44: value 10n -> 1u
- C45, C46: value 100n -> 10n
- C48: value 0.1u -> 100n
- C49: value 100p -> 1n
- C58, C67: value 100p -> 1u
- C59, C68: value 1n -> 10n
- C76: value 0.1uF -> 1u
- C77: value 0.1uF -> 10n
- C80, C81: value 1n -> 0.1uF
- C82, C85: value 0.1u -> 1n
- C86: value 4.7u -> 1n; footprint Capacitor_SMD:C_0805_2012Metric_Pad1.18x1.45mm_HandSolder -> Capacitor_SMD:C_0603_1608Metric_Pad1.08x0.95mm_HandSolder
- C87: value 100n -> 0.1u
- C88: value 100n -> 4.7u; footprint Capacitor_SMD:C_0603_1608Metric_Pad1.08x0.95mm_HandSolder -> Capacitor_SMD:C_0805_2012Metric_Pad1.18x1.45mm_HandSolder
- C89: value 47u -> 100n; footprint Capacitor_SMD:C_1210_3225Metric_Pad1.33x2.70mm_HandSolder -> Capacitor_SMD:C_0603_1608Metric_Pad1.08x0.95mm_HandSolder
- D10: value LED -> RGB_LED; footprint LED_SMD:LED_0603_1608Metric -> LHRS_Special:RGB_LED
- D11: value D_Schottky -> TVS; footprint Diode_SMD:D_SOD-123 -> Diode_SMD:D_SOD-323
- D12: value TPD2EUSB30DRTR -> LED; footprint LHRS_ICs:TPD2EUSB30DRTR -> LED_SMD:LED_0603_1608Metric
- D5: value SMBJ30CD -> SMBJ15CA
- D8: value RGB_LED -> D_Schottky; footprint LHRS_Special:RGB_LED -> Diode_SMD:D_SOD-123
- D9: value TVS -> TPD2EUSB30DRTR; footprint Diode_SMD:D_SOD-323 -> LHRS_ICs:TPD2EUSB30DRTR
- F1: value Fuse_3557_2 -> 1A
- IC1: value TCAN3413DR -> LM74502DDFR; footprint LHRS_Passives:TCAN3413DR -> LHRS_Power:LM74502DDFR
- J6: value SWD_Header -> USB_C_Receptacle_USB2.0_16P; footprint LHRS_Connectors:SWD_Conn -> LHRS_Connectors:USB_C_Receptacle_GCT_USB4105-xx-A_16P_TopMnt_Horizontal
- J7: value SWD -> SWD_Header; footprint Connector_PinHeader_2.54mm:PinHeader_1x04_P2.54mm_Vertical -> LHRS_Connectors:SWD_Conn
- J8: value USB_C_Receptacle_USB2.0_16P -> SWD; footprint LHRS_Connectors:USB_C_Receptacle_GCT_USB4105-xx-A_16P_TopMnt_Horizontal -> Connector_PinHeader_2.54mm:PinHeader_1x04_P2.54mm_Vertical
- L1: footprint LHRS_Passives:SRN8040-150M -> LHRS_Passives:74439369082
- R10: value 10k -> 7.32k
- R11: value 10k -> 100k
- R12: value 137k -> 15.8k
- R24: value 1k -> 5.1k
- R25: value 10k -> 5.1k
- R27: value 1k -> 10k
- R28, R29: value 22 -> 1k
- R30: value 10k -> 22
- R31: value 1k -> 22
- R32: value 5.1k -> 10k
- R33: value 5.1k -> 1k
- R34: value 10k -> 0
- R37, R44: value 20k -> 10k
- R40: value 100 -> 20k
- R42: value 10k -> 100
- R46: value 10k -> 20k
- R47, R49: value 500k -> 10k; footprint Resistor_SMD:R_0805_2012Metric_Pad1.20x1.40mm_HandSolder -> Resistor_SMD:R_0603_1608Metric_Pad0.98x0.95mm_HandSolder
- R48: value 500k -> 90k; footprint Resistor_SMD:R_0805_2012Metric_Pad1.20x1.40mm_HandSolder -> Resistor_SMD:R_0603_1608Metric_Pad0.98x0.95mm_HandSolder
- R50, R57, R64: value 20k -> 500k; footprint Resistor_SMD:R_0603_1608Metric_Pad0.98x0.95mm_HandSolder -> Resistor_SMD:R_0805_2012Metric_Pad1.20x1.40mm_HandSolder
- R51, R58, R65: value 47k -> 500k; footprint Resistor_SMD:R_0603_1608Metric_Pad0.98x0.95mm_HandSolder -> Resistor_SMD:R_0805_2012Metric_Pad1.20x1.40mm_HandSolder
- R52, R59, R66: value 10 -> 500k; footprint Resistor_SMD:R_0603_1608Metric_Pad0.98x0.95mm_HandSolder -> Resistor_SMD:R_0805_2012Metric_Pad1.20x1.40mm_HandSolder
- R53, R60, R67: value 10 -> 20k
- R54, R61: value 500k -> 47k; footprint Resistor_SMD:R_0805_2012Metric_Pad1.20x1.40mm_HandSolder -> Resistor_SMD:R_0603_1608Metric_Pad0.98x0.95mm_HandSolder
- R55, R56, R62, R63: value 500k -> 10; footprint Resistor_SMD:R_0805_2012Metric_Pad1.20x1.40mm_HandSolder -> Resistor_SMD:R_0603_1608Metric_Pad0.98x0.95mm_HandSolder
- R68: value 16k -> 47k
- R69: value 4.7k -> 10
- R70: value 10k -> 10
- R71: value 10k -> 16k
- R72: value 10k -> 4.7k
- R83: value 100k -> 10k; footprint Resistor_SMD:R_0603_1608Metric -> Resistor_SMD:R_0603_1608Metric_Pad0.98x0.95mm_HandSolder
- R84: value 19.1k -> 10k; footprint Resistor_SMD:R_0603_1608Metric -> Resistor_SMD:R_0603_1608Metric_Pad0.98x0.95mm_HandSolder
- R9: value 221k -> 100k
- TP10: value PP OV -> HALL_UOUT
- TP11: value PP SOURCE -> HALL_UREF
- TP12: value PR_TP -> HALL_OCD
- TP13: value HALL_UOUT -> SHUNT_OUTN
- TP14: value HALL_UREF -> SHUNT_OUTP
- TP15: value HALL_OCD -> Scrut Vin+
- TP16: value SHUNT_OUTN -> Scrut Vout
- TP17: value SHUNT_OUTP -> Scrut Vin-
- TP18: value SHUNT_ADC -> SHUNT_Vout
- TP7: value USB_5V -> CC1
- TP8: value PP GATE -> CC2
- TP9: value PP EN -> PR_TP
- U1: value LM74502DDFR -> MCP1826S; footprint LHRS_Power:LM74502DDFR -> Package_TO_SOT_SMD:SOT-223-3_TabPin2
- U10: value AMC3311QDWERQ1 -> TPS2117DRLR; footprint AMC3311QDWERQ1:DWE0016A-IPC_A -> LHRS_Power:TPS2117DRLR
- U11: value TPS2117DRLR -> TLV9002QDRQ1; footprint LHRS_Power:TPS2117DRLR -> Package_SO:SOIC-8_3.9x4.9mm_P1.27mm
- U13: value TLV9002QDRQ1 -> LMR51635XDDCR; footprint Package_SO:SOIC-8_3.9x4.9mm_P1.27mm -> LHRS_ICs:DDC0006A-MFG
- U2: value MCP1826S -> CDSOT23-T24CAN; footprint Package_TO_SOT_SMD:SOT-223-3_TabPin2 -> LHRS_ICs:CDSOT23-T24CAN
- U4: value CDSOT23-T24CAN -> AMC3311QDWERQ1; footprint LHRS_ICs:CDSOT23-T24CAN -> AMC3311QDWERQ1:DWE0016A-IPC_A
- U5: value AMC3311QDWERQ1 -> STM32G473CETx; footprint AMC3311QDWERQ1:DWE0016A-IPC_A -> LHRS_Special:48PinMCU
- U6: value STM32G473CETx -> TLV9002QDRQ1; footprint LHRS_Special:48PinMCU -> Package_SO:SOIC-8_3.9x4.9mm_P1.27mm
- U7: value TLV9002QDRQ1 -> AMC3311QDWERQ1; footprint Package_SO:SOIC-8_3.9x4.9mm_P1.27mm -> AMC3311QDWERQ1:DWE0016A-IPC_A
- moved TP_1 195.1 mm to (222.6, 37.3)
- moved D7 180.7 mm to (207.8, 52.0), turned to 180 degrees
- moved C9 162.3 mm to (214.3, 59.5), turned to 180 degrees
- moved C8 160.3 mm to (213.9, 49.7), turned to 180 degrees
- moved TP7 159.8 mm to (222.5, 31.6)
- moved R34 158.3 mm to (178.7, 49.7)
- moved TP8 157.8 mm to (217.7, 31.6)
- moved U4 157.5 mm to (184.6, 84.7)
- moved C25 153.9 mm to (178.4, 113.3)
- moved C26 153.9 mm to (178.4, 115.9)
- moved C7 152.4 mm to (183.0, 36.2), turned to -90 degrees
- moved TP40 151.6 mm to (222.8, 42.8)
- moved TP41 149.2 mm to (220.2, 47.5)
- moved TP9 148.5 mm to (217.7, 37.3)
- moved TP39 145.4 mm to (217.8, 42.7)
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Connections:
- C11 pad 1: Net-(C11-Pad1) -> /+3v3
- C13 pad 1: /+3v3 -> Net-(C13-Pad1)
- C15 pad 1: Net-(C15-Pad1) -> /+3v3
- C16 pad 1: Net-(U5-IN) -> /+3v3
- C16 pad 2: HV GND -> GND
- C17 pad 1: Net-(U5-DCDC_OUT) -> Net-(C17-Pad1)
- C17 pad 2: HV GND -> GND
- C18 pad 1: HV GND -> Net-(U4-IN)
- C18 pad 2: Net-(U5-DCDC_OUT) -> HV GND
- C19 pad 1: HV GND -> Net-(U4-DCDC_OUT)
- C19 pad 2: Net-(U5-HLDO_OUT) -> HV GND
- C20 pad 2: Net-(U5-HLDO_OUT) -> Net-(U4-DCDC_OUT)
- C21 pad 1: Net-(U5-DCDC_IN) -> HV GND
- C21 pad 2: GND -> Net-(U4-HLDO_OUT)
- C22 pad 1: /+3v3 -> HV GND
- C22 pad 2: GND -> Net-(U4-HLDO_OUT)
- C23 pad 1: /+3v3 -> Net-(U4-DCDC_IN)
- C24 pad 1: /Voltage_Sense/HV-_N -> /+3v3
- C24 pad 2: /Voltage_Sense/HV-_P -> GND
- C25 pad 1: GND -> /+3v3
- C25 pad 2: Net-(U6-PF0-OSC_IN) -> GND
- C26 pad 1: Net-(U6-PF1-OSC_OUT) -> /Voltage_Sense/HV-_N
- C26 pad 2: GND -> /Voltage_Sense/HV-_P
- C27 pad 1: /+3v3 -> GND
- C27 pad 2: GND -> /Power_Data/Power_Mux/VIN_1
- C28 pad 1: /48PinMCU/VDDA -> GND
- C28 pad 2: /48PinMCU/GNDA -> Net-(U5-PF0-OSC_IN)
- C29 pad 1: /48PinMCU/NRST -> Net-(U5-PF1-OSC_OUT)
- C3 pad 2: Net-(U1-VCAP) -> Net-(IC1-VCAP)
- C32 pad 1: /+3v3 -> /48PinMCU/NRST
- C33 pad 1: /48PinMCU/VDDA -> /+3v3
- C33 pad 2: /48PinMCU/GNDA -> GND
- C34 pad 1: /+3v3 -> /48PinMCU/VDDA
- C34 pad 2: GND -> /48PinMCU/GNDA
- C35 pad 1: /48PinMCU/VDDA -> /+3v3
- C35 pad 2: /48PinMCU/GNDA -> GND
- C36 pad 1: /+3v3 -> /48PinMCU/VDDA
- C36 pad 2: GND -> /48PinMCU/GNDA
- C38 pad 1: /+3v3 -> /48PinMCU/VDDA
- C38 pad 2: GND -> /48PinMCU/GNDA
- C39 pad 1: /48PinMCU/VDDA -> /+3v3
- C39 pad 2: /48PinMCU/GNDA -> GND
- C40 pad 1: GND -> /+3v3
- C40 pad 2: /Power_Data/USB_5V -> GND
- C41 pad 1: /+5V -> /+3v3
- C42 pad 1: /+5V -> /48PinMCU/VDDA
- C42 pad 2: GND -> /48PinMCU/GNDA
- C43 pad 1: /HALL_UOUT -> /+5V
- C44 pad 1: /HALL_UREF -> /+5V
- C45 pad 1: Net-(C45-Pad1) -> /HALL_UOUT
- C45 pad 2: Net-(C45-Pad2) -> GND
- C46 pad 1: /SHUNT_UREF -> /HALL_UREF
- C47 pad 1: Net-(U7B--) -> Net-(C47-Pad1)
- C47 pad 2: Net-(U7A--) -> Net-(C47-Pad2)
- C48 pad 1: /+3v3 -> /SHUNT_UREF
- C49 pad 1: Net-(U8-IN) -> /Current_Sense/SHUNT Vout
- C49 pad 2: HV GND -> Net-(U6A--)
- C50 pad 1: Net-(U8-DCDC_OUT) -> /+3v3
- C50 pad 2: HV GND -> GND
- C51 pad 1: HV GND -> Net-(U7-IN)
- C51 pad 2: Net-(U8-DCDC_OUT) -> HV GND
- C52 pad 1: HV GND -> Net-(U7-DCDC_OUT)
- C52 pad 2: Net-(U8-HLDO_OUT) -> HV GND
- C53 pad 2: Net-(U8-HLDO_OUT) -> Net-(U7-DCDC_OUT)
- C54 pad 1: Net-(U8-DCDC_IN) -> HV GND
- C54 pad 2: GND -> Net-(U7-HLDO_OUT)
- C55 pad 1: /+3v3 -> HV GND
- C55 pad 2: GND -> Net-(U7-HLDO_OUT)
- C56 pad 1: /+3v3 -> Net-(U7-DCDC_IN)
- C57 pad 1: /Voltage_Sense/Motor-_N -> /+3v3
- C57 pad 2: /Voltage_Sense/Motor-_P -> GND
- C58 pad 1: Net-(U9-IN) -> /+3v3
- C58 pad 2: HV GND -> GND
- C59 pad 1: Net-(U9-DCDC_OUT) -> /Voltage_Sense/Motor-_N
- C59 pad 2: HV GND -> /Voltage_Sense/Motor-_P
- C6 pad 2: Net-(D7-K) -> /Power_Data/PowerProtection/OV
- C60 pad 1: HV GND -> Net-(U8-IN)
- C60 pad 2: Net-(U9-DCDC_OUT) -> HV GND
- C61 pad 1: HV GND -> Net-(U8-DCDC_OUT)
- C61 pad 2: Net-(U9-HLDO_OUT) -> HV GND
- C62 pad 2: Net-(U9-HLDO_OUT) -> Net-(U8-DCDC_OUT)
- C63 pad 1: Net-(U9-DCDC_IN) -> HV GND
- C63 pad 2: GND -> Net-(U8-HLDO_OUT)
- C64 pad 1: /+3v3 -> HV GND
- C64 pad 2: GND -> Net-(U8-HLDO_OUT)
- C65 pad 1: /+3v3 -> Net-(U8-DCDC_IN)
- C66 pad 1: /Voltage_Sense/HV+_N -> /+3v3
- C66 pad 2: /Voltage_Sense/HV+_P -> GND
- C67 pad 1: Net-(U10-IN) -> /+3v3
- C67 pad 2: HV GND -> GND
- C68 pad 1: Net-(U10-DCDC_OUT) -> /Voltage_Sense/HV+_N
- C68 pad 2: HV GND -> /Voltage_Sense/HV+_P
- C69 pad 1: HV GND -> Net-(U9-IN)
- C69 pad 2: Net-(U10-DCDC_OUT) -> HV GND
- C7 pad 2: /+3v3 -> /Power_Data/PowerProtection/EN/UVLO
- C70 pad 1: HV GND -> Net-(U9-DCDC_OUT)
- C70 pad 2: Net-(U10-HLDO_OUT) -> HV GND
- C71 pad 2: Net-(U10-HLDO_OUT) -> Net-(U9-DCDC_OUT)
- C72 pad 1: Net-(U10-DCDC_IN) -> HV GND
- C72 pad 2: GND -> Net-(U9-HLDO_OUT)
- C73 pad 1: /+3v3 -> HV GND
- C73 pad 2: GND -> Net-(U9-HLDO_OUT)
- C74 pad 1: /+3v3 -> Net-(U9-DCDC_IN)
- C75 pad 1: /Voltage_Sense/Motor+_N -> /+3v3
- C75 pad 2: /Voltage_Sense/Motor+_P -> GND
- C76 pad 1: /Power_Data/USB_5V -> /+3v3
- C77 pad 1: /Power_Data/Buck_5V -> /Voltage_Sense/Motor+_N
- C77 pad 2: GND -> /Voltage_Sense/Motor+_P
- C78 pad 1: /Power_Data/Power_Mux/PR1 -> /Power_Data/Power_Mux/VIN_1
- C79 pad 1: /+5V -> /Power_Data/Buck_5V
- C8 pad 1: /+3v3 -> GND
- C8 pad 2: GND -> Net-(D7-K)
- C80 pad 1: Net-(U12A--) -> /Power_Data/Power_Mux/PR1
- C80 pad 2: /MOTOR+_ADC -> GND
- C81 pad 1: Net-(U12B--) -> /+5V
- C81 pad 2: /HV+_ADC -> GND
- C82 pad 1: /+3v3 -> Net-(U11A--)
- C82 pad 2: GND -> /MOTOR+_ADC
- C83 pad 1: Net-(U13A--) -> Net-(U11B--)
- C83 pad 2: /HV-_ADC -> /HV+_ADC
- C84 pad 1: Net-(U13B--) -> /+3v3
- C84 pad 2: /MOTOR-_ADC -> GND
- C85 pad 1: /+3v3 -> Net-(U12A--)
- C85 pad 2: GND -> /HV-_ADC
- C86 pad 1: /+12V -> Net-(U12B--)
- C86 pad 2: GND -> /MOTOR-_ADC
- C87 pad 1: /+12V -> /+3v3
- C88 pad 1: /Power_Data/12VBuck/CB -> /+12V
- C88 pad 2: /Power_Data/12VBuck/SW -> GND
- C89 pad 1: /Power_Data/Buck_5V -> /+12V
- C9 pad 1: /+3v3 -> GND
- C9 pad 2: GND -> /+3v3
- D10 pad 1: Net-(D10-K) -> /48PinMCU/PA2
- D10 pad 2: Net-(D10-A) -> Net-(D10-Pad2)
- D11 pad 1: /Power_Data/USB_5V -> GND
- D11 pad 2: /Power_Data/VBUS_IN -> Net-(D11-A2)
- D12 pad 1: /USB_DP -> Net-(D12-K)
- D12 pad 2: /USB_DM -> Net-(D11-A2)
- D17 pad 2: /SHUNT_UOUT -> /Current_Sense/SHUNT Vout
- D18 pad 1: /SHUNT_UOUT -> /Current_Sense/SHUNT Vout
- D5 pad 1: /+12V_Ext -> GND
- D5 pad 2: GND -> /+12V_Ext
- D8 pad 1: /48PinMCU/PA2 -> /Power_Data/Power_Mux/VIN_1
- D8 pad 2: Net-(D8-Pad2) -> /Power_Data/USB-C Connector/VBUS_IN
- D9 pad 1: GND -> /USB_DP
- D9 pad 2: Net-(D10-A) -> /USB_DM
- IC1 pad 1: /CAN2_TX -> /Power_Data/PowerProtection/EN/UVLO
- IC1 pad 3: /+3v3 -> unconnected-(IC1-N.C-Pad3)
- IC1 pad 4: /CAN2_RX -> Net-(IC1-VCAP)
- IC1 pad 5: /+3v3 -> Net-(D6-K)
- IC1 pad 6: /BPS_CAN_L -> /Power_Data/PowerProtection/gate
- IC1 pad 7: /BPS_CAN_H -> /Power_Data/PowerProtection/OV
- IC1 pad 8: GND -> /Power_Data/PowerProtection/source
- IC2 pad 1: /CAN1_TX -> /CAN2_TX
- IC2 pad 4: /CAN1_RX -> /CAN2_RX
- IC2 pad 6: /IMD_CAN_L -> /BPS_CAN_L
- IC2 pad 7: /IMD_CAN_H -> /BPS_CAN_H
- J7 pad 3: Net-(J6-Pin_3) -> Net-(J7-Pin_3)
- J7 pad 4: Net-(J6-Pin_4) -> Net-(J7-Pin_4)
- R11 pad 1: /Power_Data/PowerProtection/EN/UVLO -> /+12V_Ext
- R11 pad 2: GND -> /Power_Data/PowerProtection/EN/UVLO
- R12 pad 1: /Power_Data/PowerProtection/EN/UVLO -> GND
- R12 pad 2: /+12V_Ext -> /Power_Data/PowerProtection/EN/UVLO
- R13 pad 2: Net-(C11-Pad1) -> Net-(C13-Pad1)
- R14 pad 1: Net-(C11-Pad1) -> Net-(C13-Pad1)
- R15 pad 2: Net-(C15-Pad1) -> Net-(C17-Pad1)
- R16 pad 1: Net-(C15-Pad1) -> Net-(C17-Pad1)
- R19 pad 2: Net-(U5-IN) -> Net-(U4-IN)
- R20 pad 2: Net-(U5-IN) -> Net-(U4-IN)
- R22 pad 1: Net-(U5-OUTP) -> Net-(U4-OUTP)
- R23 pad 1: Net-(U5-OUTN) -> Net-(U4-OUTN)
- R24 pad 1: Net-(D8-Pad2) -> GND
- R24 pad 2: GND -> /Power_Data/USB-C Connector/CC1
- R25 pad 1: /48PinMCU/NRST -> GND
- R25 pad 2: /+3v3 -> /Power_Data/USB-C Connector/CC2
- R26 pad 1: Net-(D8-Pad4) -> Net-(D10-Pad2)
- R27 pad 1: Net-(D8-Pad6) -> /48PinMCU/NRST
- R27 pad 2: GND -> /+3v3
- R28 pad 1: /48PinMCU/SWCLK -> Net-(D10-Pad4)
- R28 pad 2: Net-(J6-Pin_3) -> GND
- R29 pad 1: /48PinMCU/SWDIO -> Net-(D10-Pad6)
- R29 pad 2: Net-(J6-Pin_4) -> GND
- R30 pad 1: /48PinMCU/BOOT0 -> /48PinMCU/SWCLK
- R30 pad 2: Net-(D10-A) -> Net-(J7-Pin_3)
- R31 pad 1: Net-(D10-K) -> /48PinMCU/SWDIO
- R31 pad 2: GND -> Net-(J7-Pin_4)
- R32 pad 1: GND -> /48PinMCU/BOOT0
- R32 pad 2: /Power_Data/CC1 -> Net-(D11-A2)
- R33 pad 1: GND -> Net-(D12-K)
- R33 pad 2: /Power_Data/CC2 -> GND
- R34 pad 1: /HALL_UOUT -> /+12V_Ext
- R34 pad 2: /Current_Sense/LZSR_UOUT -> /+12V
- R35 pad 1: /HALL_UREF -> /HALL_UOUT
- R35 pad 2: /Current_Sense/LZSR_UREF -> /Current_Sense/LZSR_UOUT
- R36 pad 1: /HALL_OCD -> /HALL_UREF
- R36 pad 2: /Current_Sense/LZSR_OCD -> /Current_Sense/LZSR_UREF
- R37 pad 2: /+3v3 -> /Current_Sense/LZSR_OCD
- R38 pad 1: GND -> /HALL_OCD
- R38 pad 2: /HALL_UOUT -> /+3v3
- R39 pad 2: /HALL_UREF -> /HALL_UOUT
- R40 pad 1: Net-(C45-Pad1) -> GND
- R40 pad 2: Net-(J10-Out-) -> /HALL_UREF
- R41 pad 1: Net-(C45-Pad2) -> Net-(C47-Pad1)
- R41 pad 2: Net-(J10-Out+) -> Net-(J10-Out-)
- R42 pad 1: Net-(U7A--) -> Net-(C47-Pad2)
- R42 pad 2: Net-(C45-Pad1) -> Net-(J10-Out+)
- R43 pad 1: /SHUNT_UREF -> Net-(U6A--)
- R43 pad 2: Net-(C45-Pad2) -> Net-(C47-Pad1)
- R44 pad 2: /+3v3 -> Net-(C47-Pad2)
- R45 pad 2: GND -> /+3v3
- R46 pad 1: Net-(U7B--) -> /SHUNT_UREF
- R46 pad 2: Net-(U7A--) -> GND
- R47 pad 1: /Motor_Precharge- -> /Current_Sense/SHUNT Vout
- R47 pad 2: Net-(R47-Pad2) -> Net-(U6A--)
- R48 pad 1: Net-(R47-Pad2) -> /Current_Sense/Vin+
- R48 pad 2: Net-(R48-Pad2) -> /Current_Sense/Scrut Vout
- R49 pad 1: Net-(R48-Pad2) -> /Current_Sense/Scrut Vout
- R49 pad 2: Net-(U8-IN) -> /Current_Sense/Vin-
- R50 pad 1: HV GND -> /Motor_Precharge-
- R50 pad 2: Net-(U8-IN) -> Net-(R50-Pad2)
- R51 pad 1: /+3v3 -> Net-(R50-Pad2)
- R51 pad 2: /MOTOR-_DIAG -> Net-(R51-Pad2)
- R52 pad 1: Net-(U8-OUTP) -> Net-(R51-Pad2)
- R52 pad 2: /Voltage_Sense/Motor-_P -> Net-(U7-IN)
- R53 pad 1: Net-(U8-OUTN) -> HV GND
- R53 pad 2: /Voltage_Sense/Motor-_N -> Net-(U7-IN)
- R54 pad 1: /HV+ -> /+3v3
- R54 pad 2: Net-(R54-Pad2) -> /MOTOR-_DIAG
- R55 pad 1: Net-(R54-Pad2) -> Net-(U7-OUTP)
- R55 pad 2: Net-(R55-Pad2) -> /Voltage_Sense/Motor-_P
- R56 pad 1: Net-(R55-Pad2) -> Net-(U7-OUTN)
- R56 pad 2: Net-(U9-IN) -> /Voltage_Sense/Motor-_N
- R57 pad 1: HV GND -> /HV+
- R57 pad 2: Net-(U9-IN) -> Net-(R57-Pad2)
- R58 pad 1: /+3v3 -> Net-(R57-Pad2)
- R58 pad 2: /HV+_DIAG -> Net-(R58-Pad2)
- R59 pad 1: Net-(U9-OUTP) -> Net-(R58-Pad2)
- R59 pad 2: /Voltage_Sense/HV+_P -> Net-(U8-IN)
- R60 pad 1: Net-(U9-OUTN) -> HV GND
- R60 pad 2: /Voltage_Sense/HV+_N -> Net-(U8-IN)
- R61 pad 1: /Motor_Precharge+ -> /+3v3
- R61 pad 2: Net-(R61-Pad2) -> /HV+_DIAG
- R62 pad 1: Net-(R61-Pad2) -> Net-(U8-OUTP)
- R62 pad 2: Net-(R62-Pad2) -> /Voltage_Sense/HV+_P
- R63 pad 1: Net-(R62-Pad2) -> Net-(U8-OUTN)
- R63 pad 2: Net-(U10-IN) -> /Voltage_Sense/HV+_N
- R64 pad 1: HV GND -> /Motor_Precharge+
- R64 pad 2: Net-(U10-IN) -> Net-(R64-Pad2)
- R65 pad 1: /+3v3 -> Net-(R64-Pad2)
- R65 pad 2: /MOTOR+_DIAG -> Net-(R65-Pad2)
- R66 pad 1: Net-(U10-OUTP) -> Net-(R65-Pad2)
- R66 pad 2: /Voltage_Sense/Motor+_P -> Net-(U9-IN)
- R67 pad 1: Net-(U10-OUTN) -> HV GND
- R67 pad 2: /Voltage_Sense/Motor+_N -> Net-(U9-IN)
- R68 pad 1: /Power_Data/USB_5V -> /+3v3
- R68 pad 2: /Power_Data/Power_Mux/PR1 -> /MOTOR+_DIAG
- R69 pad 1: /Power_Data/Power_Mux/PR1 -> Net-(U9-OUTP)
- R69 pad 2: GND -> /Voltage_Sense/Motor+_P
- R70 pad 1: /Power_Data/USB_5V -> Net-(U9-OUTN)
- R70 pad 2: Net-(U11-ST) -> /Voltage_Sense/Motor+_N
- R71 pad 1: /Voltage_Sense/HV+_P -> /Power_Data/Power_Mux/VIN_1
- R71 pad 2: Net-(U12A-+) -> /Power_Data/Power_Mux/PR1
- R72 pad 1: /Voltage_Sense/HV+_N -> /Power_Data/Power_Mux/PR1
- R72 pad 2: Net-(U12A--) -> GND
- R73 pad 1: /Voltage_Sense/HV-_P -> /Power_Data/Power_Mux/VIN_1
- R73 pad 2: Net-(U12B-+) -> Net-(U10-ST)
- R74 pad 1: /Voltage_Sense/HV-_N -> /Voltage_Sense/HV+_P
- R74 pad 2: Net-(U12B--) -> Net-(U11A-+)
- R75 pad 1: /MOTOR+_ADC -> /Voltage_Sense/HV+_N
- R75 pad 2: Net-(U12A--) -> Net-(U11A--)
- R76 pad 1: /HV+_ADC -> /Voltage_Sense/HV-_P
- R76 pad 2: Net-(U12B--) -> Net-(U11B-+)
- R77 pad 1: /Voltage_Sense/Motor+_P -> /Voltage_Sense/HV-_N
- R77 pad 2: Net-(U13A-+) -> Net-(U11B--)
- R78 pad 1: /Voltage_Sense/Motor+_N -> /MOTOR+_ADC
- R78 pad 2: Net-(U13A--) -> Net-(U11A--)
- R79 pad 1: /Voltage_Sense/Motor-_P -> /HV+_ADC
- R79 pad 2: Net-(U13B-+) -> Net-(U11B--)
- R80 pad 1: /Voltage_Sense/Motor-_N -> /Voltage_Sense/Motor+_P
- R80 pad 2: Net-(U13B--) -> Net-(U12A-+)
- R81 pad 1: /HV-_ADC -> /Voltage_Sense/Motor+_N
- R81 pad 2: Net-(U13A--) -> Net-(U12A--)
- R82 pad 1: /MOTOR-_ADC -> /Voltage_Sense/Motor-_P
- R82 pad 2: Net-(U13B--) -> Net-(U12B-+)
- R83 pad 1: /Power_Data/Buck_5V -> /Voltage_Sense/Motor-_N
- R83 pad 2: /Power_Data/12VBuck/FB -> Net-(U12B--)
- R84 pad 1: /Power_Data/12VBuck/FB -> /HV-_ADC
- R84 pad 2: GND -> Net-(U12A--)
- SW2 pad 2: Net-(D10-A) -> Net-(D11-A2)
- TP10 pad 1: /Power_Data/PowerProtection/OV -> /Current_Sense/LZSR_UOUT
- TP11 pad 1: /Power_Data/PowerProtection/source -> /Current_Sense/LZSR_UREF
- TP12 pad 1: /Power_Data/Power_Mux/PR1 -> /Current_Sense/LZSR_OCD
- TP13 pad 1: /Current_Sense/LZSR_UOUT -> Net-(U6A--)
- TP14 pad 1: /Current_Sense/LZSR_UREF -> /SHUNT_UREF
- TP15 pad 1: /Current_Sense/LZSR_OCD -> /Current_Sense/Vin+
- TP16 pad 1: Net-(U7A--) -> /Current_Sense/Scrut Vout
- TP17 pad 1: /SHUNT_UREF -> /Current_Sense/Vin-
- TP18 pad 1: /SHUNT_UOUT -> /Current_Sense/SHUNT Vout
- TP7 pad 1: /Power_Data/USB_5V -> /Power_Data/USB-C Connector/CC1
- TP8 pad 1: /Power_Data/PowerProtection/gate -> /Power_Data/USB-C Connector/CC2
- TP9 pad 1: /Power_Data/PowerProtection/EN/UVLO -> /Power_Data/Power_Mux/PR1
- U1 pad 1: /Power_Data/PowerProtection/EN/UVLO -> Net-(D7-K)
- U1 pad 3: unconnected-(U1-N.C-Pad3) -> /+3v3
- U10 pad 1: Net-(U10-DCDC_OUT) -> GND
- U10 pad 2: HV GND -> /+5V
- U10 pad 3: Net-(U10-DCDC_OUT) -> /Power_Data/Power_Mux/VIN_1
- U10 pad 4: unconnected-(U10-NC-Pad4) -> /Power_Data/Power_Mux/PR1
- U10 pad 5: Net-(U10-HLDO_OUT) -> /Power_Data/Power_Mux/VIN_1
- U10 pad 6: Net-(U10-IN) -> /Power_Data/Buck_5V
- U10 pad 7: HV GND -> /+5V
- U10 pad 8: HV GND -> Net-(U10-ST)
- U11 pad 1: GND -> /MOTOR+_ADC
- U11 pad 2: /+5V -> Net-(U11A--)
- U11 pad 3: /Power_Data/USB_5V -> Net-(U11A-+)
- U11 pad 4: /Power_Data/Power_Mux/PR1 -> GND
- U11 pad 5: /Power_Data/USB_5V -> Net-(U11B-+)
- U11 pad 6: /Power_Data/Buck_5V -> Net-(U11B--)
- U11 pad 7: /+5V -> /HV+_ADC
- U11 pad 8: Net-(U11-ST) -> /+3v3
- U12 pad 1: /MOTOR+_ADC -> /HV-_ADC
- U12 pad 7: /HV+_ADC -> /MOTOR-_ADC
- U13 pad 1: /HV-_ADC -> /Power_Data/12VBuck/FB
- U13 pad 2: Net-(U13A--) -> /+12V
- U13 pad 3: Net-(U13A-+) -> /+12V
- U13 pad 5: Net-(U13B-+) -> /Power_Data/12VBuck/SW
- U13 pad 6: Net-(U13B--) -> /Power_Data/12VBuck/CB
- U2 pad 1: Net-(D7-K) -> /BPS_CAN_H
- U2 pad 2: GND -> /BPS_CAN_L
- U2 pad 3: /+3v3 -> GND
- U3 pad 1: /BPS_CAN_H -> /IMD_CAN_H
- U3 pad 2: /BPS_CAN_L -> /IMD_CAN_L
- U4 pad 1: /IMD_CAN_H -> Net-(U4-DCDC_OUT)
- U4 pad 2: /IMD_CAN_L -> HV GND
- U4 pad 3: GND -> Net-(U4-DCDC_OUT)
- U5 pad 1: Net-(U5-DCDC_OUT) -> /+3v3
- U5 pad 10: Net-(U5-OUTN) -> /48PinMCU/PA2
- U5 pad 11: Net-(U5-OUTP) -> /SHUNT_UOUT
- U5 pad 12: /+3v3 -> /SHUNT_UREF
- U5 pad 13: Net-(U5-DCDC_IN) -> /HV+_DIAG
- U5 pad 14: /HV-_DIAG -> /HV+_ADC
- U5 pad 15: GND -> /HV-_ADC
- U5 pad 16: Net-(U5-DCDC_IN) -> /HV-_DIAG
- U5 pad 2: HV GND -> /48PinMCU/PC13
- U5 pad 3: Net-(U5-DCDC_OUT) -> /48PinMCU/PC14
- U5 pad 4: unconnected-(U5-NC-Pad4) -> /48PinMCU/PC15
- U5 pad 5: Net-(U5-HLDO_OUT) -> Net-(U5-PF0-OSC_IN)
- U5 pad 6: Net-(U5-IN) -> Net-(U5-PF1-OSC_OUT)
- U5 pad 7: HV GND -> /48PinMCU/NRST
- U5 pad 8: HV GND -> /48PinMCU/PA0
- U5 pad 9: GND -> /48PinMCU/PA1
- U6 pad 1: /+3v3 -> /Current_Sense/SHUNT Vout
- U6 pad 2: /48PinMCU/PC13 -> Net-(U6A--)
- U6 pad 3: /48PinMCU/PC14 -> /SHUNT_UREF
- U6 pad 4: /48PinMCU/PC15 -> GND
- U6 pad 5: Net-(U6-PF0-OSC_IN) -> /SHUNT_UREF
- U6 pad 6: Net-(U6-PF1-OSC_OUT) -> /Current_Sense/Vin-
- U6 pad 7: /48PinMCU/NRST -> /Current_Sense/Vin-
- U6 pad 8: /48PinMCU/PA0 -> /+3v3
- U7 pad 1: Net-(U7B--) -> Net-(U7-DCDC_OUT)
- U7 pad 2: Net-(U7A--) -> HV GND
- U7 pad 3: /SHUNT_UREF -> Net-(U7-DCDC_OUT)
- U7 pad 4: GND -> unconnected-(U7-NC-Pad4)
- U7 pad 5: /SHUNT_UOUT -> Net-(U7-HLDO_OUT)
- U7 pad 6: Net-(U7B--) -> Net-(U7-IN)
- U7 pad 7: /SHUNT_UOUT -> HV GND
- U7 pad 8: /+3v3 -> HV GND
- U8 pad 14: /MOTOR-_DIAG -> /HV+_DIAG
- U9 pad 14: /HV+_DIAG -> /MOTOR+_DIAG
- Y1 pad 1: Net-(U6-PF0-OSC_IN) -> Net-(U5-PF0-OSC_IN)
- Y1 pad 2: Net-(U6-PF1-OSC_OUT) -> Net-(U5-PF1-OSC_OUT)

Commit message: CAN stufff
Parts:
- removed the TP34 at (126.0, 72.5)
- added TP27: Motor- IN, TestPoint:TestPoint_THTPad_D3.0mm_Drill1.5mm, F.Cu at (126.2, 100.3)
- added TP38: Motor- ADC, TestPoint:TestPoint_THTPad_D3.0mm_Drill1.5mm, F.Cu at (212.7, 154.1)
- J1: value Shunt Breakout Conn -> Shunt Breakout
- J10: value SSA-2-100A -> Shunt Conn
- J2: value Hall Breakout Conn -> Hall Breakout
- TP26: value MOTOR+ DIAG -> Motor+ DIAG
- TP35: value OUT_ADC_TP -> HV- ADC
- TP36: value OUT_ADC_TP -> HV+ ADC
- TP37: value OUT_ADC_TP -> Motor+ ADC
- moved D13 180.2 mm to (206.2, 35.0)
- moved C47 175.5 mm to (205.6, 55.9), turned to 90 degrees
- moved C45 174.6 mm to (205.7, 32.9)
- moved D14 174.1 mm to (200.2, 35.0)
- moved R41 173.5 mm to (208.3, 57.0)
- moved R42 173.1 mm to (208.3, 54.8)
- moved D18 172.0 mm to (196.8, 66.2)
- moved C48 170.7 mm to (201.4, 50.8), turned to 90 degrees
- moved R39 170.4 mm to (205.8, 37.1), turned to 180 degrees
- moved J10 169.0 mm to (213.3, 48.2)
- moved J12 168.8 mm to (214.1, 74.2)
- moved C46 168.6 mm to (199.6, 32.9)
- moved D17 168.4 mm to (193.9, 56.5), turned to -90 degrees
- moved R35 168.3 mm to (203.7, 31.1), turned to 180 degrees
- moved D15 166.9 mm to (193.1, 38.0)
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- renumbered TP27 to TP28, TP28 to TP29, TP29 to TP30, TP30 to TP31, TP31 to TP32, TP32 to TP33, TP33 to TP34, TP38 to TP39, TP39 to TP40, TP40 to TP41, TP41 to TP42
Connections:
- C82 pad 2: /MOTOR+_ADC -> /HV+_ADC
- C83 pad 2: /HV+_ADC -> /HV-_ADC
- C85 pad 2: /HV-_ADC -> /MOTOR+_ADC
- D19 pad 2: /HV+_ADC -> /HV-_ADC
- D20 pad 1: /HV+_ADC -> /HV-_ADC
- D21 pad 2: /MOTOR+_ADC -> /HV+_ADC
- D22 pad 1: /MOTOR+_ADC -> /HV+_ADC
- D25 pad 2: /HV-_ADC -> /MOTOR+_ADC
- D26 pad 1: /HV-_ADC -> /MOTOR+_ADC
- R78 pad 1: /MOTOR+_ADC -> /HV+_ADC
- R79 pad 1: /HV+_ADC -> /HV-_ADC
- R84 pad 1: /HV-_ADC -> /MOTOR+_ADC
- TP35 pad 1: /MOTOR+_ADC -> /HV-_ADC
- TP36 pad 1: /MOTOR-_ADC -> /HV+_ADC
- TP37 pad 1: /HV-_ADC -> /MOTOR+_ADC
- U11 pad 1: /MOTOR+_ADC -> /HV+_ADC
- U11 pad 7: /HV+_ADC -> /HV-_ADC
- U12 pad 1: /HV-_ADC -> /MOTOR+_ADC

Commit message: saving
Parts:
- moved TP11 142.1 mm to (211.8, 29.5)
- moved C34 141.7 mm to (166.0, 65.1), turned to 180 degrees
- moved C31 140.5 mm to (166.1, 71.3), turned to 180 degrees
- moved TP14 138.8 mm to (213.1, 43.8)
- moved C37 137.0 mm to (166.1, 61.7)
- moved C38 136.4 mm to (166.1, 69.9), turned to 180 degrees
- moved C36 136.3 mm to (166.1, 68.3), turned to 180 degrees
- moved TP18 136.2 mm to (213.6, 50.0)
- moved C29 133.7 mm to (159.3, 75.6)
- moved C32 133.2 mm to (156.8, 55.8), turned to 90 degrees
- moved FB2 132.7 mm to (166.1, 63.4), turned to 180 degrees
- moved C41 132.3 mm to (166.1, 60.0)
- moved C42 132.0 mm to (166.1, 66.7), turned to 180 degrees
- moved R26 131.7 mm to (165.8, 74.0), turned to -90 degrees
- moved FB1 129.8 mm to (163.5, 63.5), turned to 90 degrees
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
Commit message: horizontal HV
Parts:
- moved TP10 118.7 mm to (154.3, 160.4)
- moved TP18 118.7 mm to (164.3, 158.0)
- moved TP11 118.7 mm to (162.6, 137.4)
- moved TP12 118.7 mm to (163.2, 143.6)
- moved TP13 118.7 mm to (164.3, 164.2)
- moved TP14 118.7 mm to (163.8, 151.7)
- moved TP31 95.4 mm to (136.6, 164.4)
- moved TP23 95.4 mm to (136.8, 156.9)
- moved D2 86.2 mm to (180.3, 40.0)
- moved R2 82.4 mm to (181.2, 42.7), turned to 90 degrees
- moved D3 81.7 mm to (176.6, 54.6), turned to 180 degrees
- moved R3 74.0 mm to (173.2, 54.6)
- moved D1 52.9 mm to (147.4, 42.5), turned to 180 degrees
- moved R1 46.1 mm to (144.7, 41.6), turned to -90 degrees
- moved J9 14.1 mm to (207.7, 27.4), turned to 0 degrees
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