File: hardware/HV_Carrier/PS-HVCarrier.kicad_pcb (KiCad board)
At the start: 2 copper layers, 293 parts, among them IC1 LM74502DDFR, IC2 TCAN3413DR, IC3 TCAN3413DR, J1 Shunt Breakout, J10 Shunt Conn, J12 Discharge Vin, J13 Charge Vin, J2 Hall Breakout, J3 IMD_Conn, J4 Voltage Tap, J5 BPS Conn, J6 USB_C_Receptacle_USB2.0_16P, J7 SWD_Header, J8 SWD, J9 LZSR 80-P, Q1 PSMN012-100YS, Q2 PSMN012-100YS, SW1 Reset, SW2 SW_SPDT, U1 MCP1826S, U10 TPS2117DRLR, U11 TLV9002QDRQ1, U12 TLV9002QDRQ1, U13 LMR51635XDDCR, U2 CDSOT23-T24CAN, U3 CDSOT23-T24CAN, U4 AMC3311QDWERQ1, U5 STM32G473CETx, U6 TLV9002QDRQ1, U7 AMC3311QDWERQ1, U8 AMC3311QDWERQ1, U9 AMC3311QDWERQ1, Y1 Crystal

Commit message: saving
Parts:
- moved TP40 121.7 mm to (50.3, 80.7)
- moved TP_1 121.7 mm to (78.8, 79.5)
- moved TP39 121.7 mm to (45.1, 80.7)
- moved TP41 121.7 mm to (35.0, 80.6)
- moved TP42 121.7 mm to (40.1, 80.7)
- moved TP7 121.7 mm to (61.8, 79.5)
- moved TP8 121.7 mm to (67.6, 79.5)
- moved TP9 121.7 mm to (73.6, 79.4)
- moved TP22 22.3 mm to (92.7, 78.8)
- moved TP29 22.3 mm to (100.5, 85.2)
- moved TP21 22.3 mm to (92.9, 85.5)
- moved TP30 22.3 mm to (100.4, 78.5)
- moved C91 11.5 mm to (167.9, 50.3), turned to -90 degrees
- moved J3 11.2 mm to (114.2, 70.5)
- moved R4 9.93 mm to (120.0, 50.7)
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Connections:
- net /USB_DM renamed /USB_D-
- net /USB_DP renamed /USB_D+
Routing:
- net /HALL_OCD: track 0.00 -> 19.1 mm
- net /+5V: track 0.00 -> 15.9 mm
- net /+3v3: track 0.00 -> 15.2 mm
- net Net-(J9-+UC): track 0.00 -> 15.0 mm
- net /Power_Data/PowerProtection/gate: track 0.00 -> 14.5 mm
- net /HALL_UREF: track 0.00 -> 13.6 mm
- net /Power_Data/Buck_5V: track 0.00 -> 12.9 mm
- net /Power_Data/Power_Mux/VIN_1: track 0.00 -> 12.7 mm
- net /Power_Data/USB-C Connector/CC2: track 0.00 -> 12.4 mm, vias 0 -> 2
- net /Power_Data/USB-C Connector/VBUS_IN: track 0.00 -> 11.3 mm, vias 0 -> 2
- net /+12V_Ext: track 0.00 -> 10.6 mm
- net /USB_D+: track 0.00 -> 9.87 mm
- net /USB_D-: track 0.00 -> 9.83 mm
- net /+12V: track 0.00 -> 9.35 mm
- net /SHUNT_UREF: track 0.00 -> 9.16 mm
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- added copper zone on F.Cu, net /+12V
- added copper zone on F.Cu, net /+12V_Ext
- added copper zone on F.Cu, net /+5V
- added copper zone on F.Cu, net /Power_Data/12VBuck/SW
- added copper zone on F.Cu, net /Power_Data/Buck_5V
- added copper zone on F.Cu, net /Power_Data/PowerProtection/source

Commit message: saving changes
Parts:
- moved TP16 72.1 mm to (243.2, 152.2)
- moved TP27 72.1 mm to (251.4, 152.4)
- moved TP25 44.8 mm to (67.1, 93.5)
- moved TP33 44.8 mm to (67.1, 101.3)
- moved TP30 44.8 mm to (58.1, 93.3)
- moved TP21 44.8 mm to (50.6, 100.2)
- moved TP22 44.8 mm to (50.4, 93.5)
- moved TP29 44.8 mm to (58.2, 99.9)
- moved TP15 44.7 mm to (233.6, 146.5)
- moved TP17 44.7 mm to (233.8, 153.2)
- moved R6 1.38 mm to (117.7, 42.4), turned to 90 degrees
- moved C13 0.34 mm to (132.7, 41.5)
- moved R14 0.34 mm to (132.7, 43.1)
- moved R16 0.13 mm to (124.0, 51.6)
- moved R48 0.10 mm to (180.4, 61.9)
Routing:
- net /+3v3: track 15.2 -> 64.0 mm, vias 0 -> 4
- net /BPS_CAN_H: track 0.00 -> 39.4 mm, vias 0 -> 2
- net /SHUNT_UOUT: track 0.00 -> 36.1 mm
- net /BPS_CAN_L: track 0.00 -> 33.0 mm
- net /SHUNT_UREF: track 9.16 -> 34.4 mm, vias 0 -> 1
- net /IMD_CAN_H: track 0.00 -> 21.9 mm
- net /Current_Sense/SHUNT Vout: track 0.00 -> 19.6 mm
- net HV GND: track 0.00 -> 19.3 mm
- net /IMD_CAN_L: track 0.00 -> 19.0 mm
- net GND: track 5.14 -> 17.3 mm
- net Net-(U6A--): track 0.00 -> 11.4 mm
- net Net-(U8-DCDC_OUT): track 0.00 -> 10.7 mm, vias 0 -> 2
- net Net-(U8-IN): track 0.00 -> 9.70 mm
- net /IMD_OKHS: track 0.00 -> 6.93 mm
- net Net-(U8-HLDO_OUT): track 0.00 -> 5.82 mm
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
Commit message: ready for review
Parts:
- removed TP2: +12V TP, TestPoint:TestPoint_THTPad_D3.0mm_Drill1.5mm
- removed TP6: +3v3 TP, TestPoint:TestPoint_THTPad_D3.0mm_Drill1.5mm
- moved TP4 164.1 mm to (226.9, 104.7)
- moved TP35 153.6 mm to (92.9, 70.2)
- moved TP36 148.5 mm to (98.0, 64.2)
- moved TP3 143.5 mm to (218.9, 43.4)
- moved TP10 140.7 mm to (218.6, 35.3)
- moved TP41 136.6 mm to (155.5, 16.3)
- moved TP12 132.3 mm to (218.8, 23.6)
- moved TP7 127.8 mm to (172.9, 16.3)
- moved TP42 127.7 mm to (150.3, 16.2)
- moved TP8 127.2 mm to (177.7, 15.8)
- moved TP11 121.4 mm to (218.3, 29.6)
- moved TP1 118.8 mm to (154.8, 129.8)
- moved TP13 118.5 mm to (218.6, 58.9)
- moved TP40 115.0 mm to (145.5, 16.2)
- moved TP9 113.6 mm to (167.9, 16.0)
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Routing:
- net /+3v3: track 64.0 -> 353.2 mm, vias 4 -> 16
- net /HALL_UOUT: track 8.22 -> 73.4 mm, vias 0 -> 3
- net /HV+_ADC: track 0.00 -> 62.0 mm, vias 0 -> 2
- net /HALL_OCD: track 19.1 -> 80.9 mm, vias 0 -> 2
- net /HV+_DIAG: track 0.00 -> 60.3 mm, vias 0 -> 2
- net HV GND: track 19.3 -> 79.4 mm
- net /HALL_UREF: track 13.6 -> 70.2 mm, vias 0 -> 3
- net /MOTOR-_DIAG: track 0.00 -> 51.2 mm, vias 0 -> 4
- net /Current_Sense/Vin-: track 8.54 -> 58.7 mm, vias 0 -> 1
- net /Current_Sense/Vin+: track 0.00 -> 44.5 mm, vias 0 -> 1
- net /Motor_Precharge-: track 0.00 -> 40.8 mm
- net /MOTOR-_ADC: track 0.00 -> 39.7 mm, vias 0 -> 2
- net /HV-_ADC: track 0.00 -> 39.0 mm, vias 0 -> 2
- net /HV-_DIAG: track 0.00 -> 38.9 mm, vias 0 -> 2
- net /USB_D-: track 9.83 -> 47.6 mm, vias 0 -> 4
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- added copper zone on F.Cu, net /+3v3
- added copper zone on B.Cu, net GND
- added copper zone on F.Cu, net GND
- added copper zone on F.Cu, net HV GND

Commit message: missing edgecut
Parts:
- TP1: value HV GND TP -> HV GND
- TP14: value SHUNT_OUTP -> SHUNT_UREF
- TP4: value GND TP -> GND
- moved H2 212.3 mm to (198.1, 37.6)
- moved H4 174.6 mm to (198.1, 151.0)
- moved H1 125.1 mm to (73.2, 37.6)
- moved TP26 92.6 mm to (125.2, 101.4), turned to 180 degrees
- moved TP4 81.3 mm to (179.3, 38.8)
- moved TP24 74.8 mm to (151.0, 92.8)
- moved TP37 74.7 mm to (146.5, 98.2)
- moved TP34 73.4 mm to (153.3, 98.3)
- moved TP23 73.1 mm to (145.1, 92.8)
- moved TP32 59.6 mm to (168.3, 105.5)
- moved TP5 54.2 mm to (75.3, 62.4)
- moved H3 51.1 mm to (73.2, 151.0)
- moved TP38 48.5 mm to (186.1, 100.1)
- moved TP42 43.2 mm to (113.5, 38.8)
- moved TP36 42.8 mm to (75.7, 100.7)
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Routing:
- net /+12V: track 9.35 -> 66.7 mm, vias 0 -> 1
- net /Current_Sense/Scrut Vout: track 5.57 -> 50.8 mm, vias 0 -> 1
- net /MOTOR-_ADC: track 39.7 -> 78.9 mm, vias 2 -> 4
- net /Voltage_Sense/Motor-_P: track 4.00 -> 36.6 mm, vias 0 -> 2
- net /Current_Sense/SHUNT Vout: track 19.6 -> 51.9 mm, vias 0 -> 1
- net /+5V: track 15.9 -> 47.5 mm
- net Net-(U6A--): track 11.4 -> 40.5 mm, vias 0 -> 1
- net /Voltage_Sense/Motor+_N: track 3.94 -> 28.0 mm, vias 0 -> 4
- net /Voltage_Sense/HV+_N: track 3.53 -> 27.3 mm, vias 0 -> 1
- net /+3v3: track 353.2 -> 375.8 mm
- net /Power_Data/12VBuck/SW: track 1.71 -> 23.1 mm, vias 0 -> 2
- net /Voltage_Sense/Motor+_P: track 3.92 -> 24.4 mm, vias 0 -> 2
- net /Power_Data/USB-C Connector/CC1: track 6.79 -> 27.2 mm
- net /Power_Data/12VBuck/CB: track 2.18 -> 21.8 mm, vias 0 -> 2
- net /Power_Data/Power_Mux/PR1: track 3.49 -> 22.5 mm, vias 0 -> 2
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