File: hardware/HV_Carrier/12VBuck.kicad_sch (KiCad schematic)
At the start: 12 parts, among them U13 LMR51635XDDCR

Commit message: saving
Parts:
- removed C91: 47u, Capacitor_SMD:C_1210_3225Metric_Pad1.33x2.70mm_HandSolder, symbol Device:C_Small
- added C91, C92: 22u, Capacitor_SMD:C_1210_3225Metric_Pad1.33x2.70mm_HandSolder, symbol Device:C
- added C93: 3.3u, Capacitor_SMD:C_0805_2012Metric_Pad1.18x1.45mm_HandSolder, symbol Device:C
- C88: LCSC P/N (none) -> C6962403
- C89: LCSC P/N (none) -> C6666325
- C90: footprint Capacitor_SMD:C_0603_1608Metric_Pad1.08x0.95mm_HandSolder -> Capacitor_SMD:C_0603_1608Metric; LCSC P/N (none) -> C6666325
- L1: footprint LHRS_Passives:SRN8040-150M -> LHRS_Passives:74439369082
- R86: renamed from R85; LCSC P/N (none) -> C25803
- R87: renamed from R86; LCSC P/N (none) -> C844132; P/N ERA-2ARB1912X -> CRCW060319K1FKEAHP
Connections:
- net GND: now also C91.2, C92.2, C93.2
- net V_out_5V: now also C91.1, C92.1, C93.1

Commit message: saving
Parts:
- renumbered TP38 to TP39, TP39 to TP40, TP40 to TP41, TP41 to TP42
Changed lines of the file:
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@@
 		(in_pos_files yes)
 		(dnp no)
-		(property "Reference" "TP38"
+		(property "Reference" "TP39"
 			(at 229.87 123.6979 0)
 			(hide yes)
@@
 			(project "PS-HVCarrier"
 				(path "/2365a867-6254-4a7c-9718-f325e0bbac5c/904fa10a-747c-46cf-90d1-33d76069dc5d/c2b7497c-dc59-4d5a-b160-c35e8bc1c10f"
-					(reference "TP38")
+					(reference "TP39")
 					(unit 1)
 				)
@@
 		(in_pos_files yes)
 		(dnp no)
-		(property "Reference" "TP40"
+		(property "Reference" "TP41"
 			(at 242.57 123.6979 0)
 			(hide yes)
@@
 			(project "PS-HVCarrier"
 				(path "/2365a867-6254-4a7c-9718-f325e0bbac5c/904fa10a-747c-46cf-90d1-33d76069dc5d/c2b7497c-dc59-4d5a-b160-c35e8bc1c10f"
-					(reference "TP40")
+					(reference "TP41")
 					(unit 1)
 				)
@@
 		(in_pos_files yes)
 		(dnp no)
-		(property "Reference" "TP39"
+		(property "Reference" "TP40"
 			(at 229.87 136.3979 0)
 			(hide yes)
@@
 			(project "PS-HVCarrier"
 				(path "/2365a867-6254-4a7c-9718-f325e0bbac5c/904fa10a-747c-46cf-90d1-33d76069dc5d/c2b7497c-dc59-4d5a-b160-c35e8bc1c10f"
-					(reference "TP39")
+					(reference "TP40")
 					(unit 1)
 				)
@@
 		(in_pos_files yes)
 		(dnp no)
-		(property "Reference" "TP41"
+		(property "Reference" "TP42"
 			(at 242.57 136.3979 0)
 			(hide yes)
@@
 			(project "PS-HVCarrier"
 				(path "/2365a867-6254-4a7c-9718-f325e0bbac5c/904fa10a-747c-46cf-90d1-33d76069dc5d/c2b7497c-dc59-4d5a-b160-c35e8bc1c10f"
-					(reference "TP41")
-					(unit 1)
-				)
+					(reference "TP42")
+					(unit 1)
+				)
