File: hardware/HV_Carrier/48PinMCU.kicad_sch (KiCad schematic)
At the start: 34 parts, among them J7 SWD_Header, J8 SWD, SW1 Reset, SW2 SW_SPDT, U5 STM32G473CETx, Y1 Crystal

Commit message: saving
Connections:
- net USB_DM renamed USB_D-
- net USB_DP renamed USB_D+
Changed lines of the file:
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@@
 		)
 	)
-	(hierarchical_label "USB_DM"
+	(hierarchical_label "USB_D-"
 		(shape bidirectional)
 		(at 121.92 64.77 0)
@@
 		)
 	)
-	(hierarchical_label "USB_DP"
+	(hierarchical_label "USB_D+"
 		(shape bidirectional)
 		(at 121.92 67.31 0)
