File: hardware/HV_Carrier/Current_Sense.kicad_sch (KiCad schematic)
At the start: 46 parts, among them J10 SSA-2-100A, J11 SSA-2-100A, J12 Discharge Vin, J13 Charge Vin, J9 LZSR 80-P, U6 TLV9002QDRQ1

Commit message: saving
Parts:
- TP15: value Scurt Vin+ -> Scrut Vin+
- TP16: value Scurt Vout -> Scrut Vout
- TP17: value Scurt Vin- -> Scrut Vin-
- renumbered R34 to R35, R35 to R36, R36 to R37, R37 to R38, R38 to R39, R39 to R40, R40 to R41, R41 to R42, R42 to R43, R43 to R44, R44 to R45, R45 to R46, R46 to R47, R47 to R48, R48 to R49
Other:
- note added: "Discharge: Vin+ = Vin- + V_bench = 1.65V + V_bench Scurt_Vout = Vin- + (Vin+ − Vin-) × R2/(R1+R2) = 1.65V + V_bench × (10k/100k) = 1.65V + 0.1 × V_bench For 70A: 0.1 × V_bench = 0.875V V_bench = 8.75V"
- note removed: "Discharge: Vin+ = Vin- + V_bench = 1.65V + V_bench Scurt_Vout = Vin- + (Vin+ − Vin-) × R2/(R1+R2) = 1.65V + V_bench × (1k/10k) = 1.65V + 0.1 × V_bench For 70A: 0.1 × V_bench = 0.875V V_bench = 8.75V"
Changed lines of the file:
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@@
 		)
 	)
-	(text "Discharge: \nVin+ = Vin- + V_bench = 1.65V + V_bench\nScurt_Vout = Vin- + (Vin+ − Vin-) × R2/(R1+R2)\n           = 1.65V + V_bench × (1k/10k)\n           = 1.65V + 0.1 × V_bench\nFor 70A: 0.1 × V_bench = 0.875V\nV_bench = 8.75V"
+	(text "Discharge: \nVin+ = Vin- + V_bench = 1.65V + V_bench\nScurt_Vout = Vin- + (Vin+ − Vin-) × R2/(R1+R2)\n           = 1.65V + V_bench × (10k/100k)\n           = 1.65V + 0.1 × V_bench\nFor 70A: 0.1 × V_bench = 0.875V\nV_bench = 8.75V"
 		(exclude_from_sim no)
 		(at 181.102 173.99 0)
@@
 		(dnp no)
 		(fields_autoplaced yes)
-		(property "Reference" "R35"
+		(property "Reference" "R36"
 			(at 77.47 54.61 90)
 			(show_name no)
@@
 			(project "PS-HVCarrier"
 				(path "/2365a867-6254-4a7c-9718-f325e0bbac5c/c64f1e33-0c51-411c-bbbf-0af7b620c655"
-					(reference "R35")
+					(reference "R36")
 					(unit 1)
 				)
@@
 		(in_pos_files yes)
 		(dnp no)
-		(property "Reference" "R42"
+		(property "Reference" "R43"
 			(at 171.45 46.99 90)
 			(show_name no)
@@
 			(project "PS-HVCarrier"
 				(path "/2365a867-6254-4a7c-9718-f325e0bbac5c/c64f1e33-0c51-411c-bbbf-0af7b620c655"
-					(reference "R42")
+					(reference "R43")
 					(unit 1)
 				)
@@
 		(in_pos_files yes)
 		(dnp no)
-		(property "Reference" "R41"
+		(property "Reference" "R42"
 			(at 154.686 54.61 90)
 			(show_name no)
@@
 			(project "PS-HVCarrier"
 				(path "/2365a867-6254-4a7c-9718-f325e0bbac5c/c64f1e33-0c51-411c-bbbf-0af7b620c655"
-					(reference "R41")
+					(reference "R42")
 					(unit 1)
 				)
@@
 		(dnp no)
 		(fields_autoplaced yes)
-		(property "Reference" "R39"
+		(property "Reference" "R40"
 			(at 93.98 63.4999 0)
 			(show_name no)
@@
 			(project "PS-HVCarrier"
 				(path "/2365a867-6254-4a7c-9718-f325e0bbac5c/c64f1e33-0c51-411c-bbbf-0af7b620c655"
-					(reference "R39")
+					(reference "R40")
 					(unit 1)
 				)
@@
 			)
 		)
-		(property "Value" "Scurt Vin+"
+		(property "Value" "Scrut Vin+"
 			(at 179.578 137.922 0)
 			(show_name no)
@@
 		(in_pos_files yes)
 		(dnp no)
-		(property "Reference" "R43"
+		(property "Reference" "R44"
 			(at 171.45 54.61 90)
 			(show_name no)
@@
 			(project "PS-HVCarrier"
 				(path "/2365a867-6254-4a7c-9718-f325e0bbac5c/c64f1e33-0c51-411c-bbbf-0af7b620c655"
-					(reference "R43")
+					(reference "R44")
 					(unit 1)
 				)
@@
 			)
 		)
-		(property "Value" "Scurt Vout"
+		(property "Value" "Scrut Vout"
 			(at 185.42 146.558 0)
 			(show_name no)
@@
 		(dnp no)
 		(fields_autoplaced yes)
-		(property "Reference" "R48"
+		(property "Reference" "R49"
 			(at 226.06 126.9999 0)
 			(show_name no)
@@
 			(project "PS-HVCarrier"
 				(path "/2365a867-6254-4a7c-9718-f325e0bbac5c/c64f1e33-0c51-411c-bbbf-0af7b620c655"
-					(reference "R48")
+					(reference "R49")
 					(unit 1)
 				)
@@
 		(dnp no)
 		(fields_autoplaced yes)
-		(property "Reference" "R38"
+		(property "Reference" "R39"
 			(at 93.98 35.5599 0)
 			(show_name no)
@@
 			(project "PS-HVCarrier"
 				(path "/2365a867-6254-4a7c-9718-f325e0bbac5c/c64f1e33-0c51-411c-bbbf-0af7b620c655"
-					(reference "R38")
+					(reference "R39")
 					(unit 1)
 				)
@@
 		(in_pos_files yes)
 		(dnp no)
-		(property "Reference" "R37"
+		(property "Reference" "R38"
 			(at 89.916 78.74 0)
 			(show_name no)
@@
 			(project "PS-HVCarrier"
 				(path "/2365a867-6254-4a7c-9718-f325e0bbac5c/c64f1e33-0c51-411c-bbbf-0af7b620c655"
-					(reference "R37")
+					(reference "R38")
 					(unit 1)
 				)
@@
 			)
 		)
-		(property "Value" "Scurt Vin-"
+		(property "Value" "Scrut Vin-"
 			(at 192.024 137.922 0)
 			(show_name no)
@@
 		(in_pos_files yes)
 		(dnp no)
-		(property "Reference" "R44"
+		(property "Reference" "R45"
 			(at 171.45 62.23 90)
 			(show_name no)
@@
 			(project "PS-HVCarrier"
 				(path "/2365a867-6254-4a7c-9718-f325e0bbac5c/c64f1e33-0c51-411c-bbbf-0af7b620c655"
-					(reference "R44")
+					(reference "R45")
 					(unit 1)
 				)
@@
 		(in_pos_files yes)
 		(dnp no)
-		(property "Reference" "R46"
+		(property "Reference" "R47"
 			(at 189.23 40.64 90)
 			(show_name no)
@@
 			(project "PS-HVCarrier"
 				(path "/2365a867-6254-4a7c-9718-f325e0bbac5c/c64f1e33-0c51-411c-bbbf-0af7b620c655"
-					(reference "R46")
+					(reference "R47")
 					(unit 1)
 				)
@@
 		(in_pos_files yes)
 		(dnp no)
-		(property "Reference" "R45"
+		(property "Reference" "R46"
 			(at 182.88 62.23 90)
 			(show_name no)
@@
 			(project "PS-HVCarrier"
 				(path "/2365a867-6254-4a7c-9718-f325e0bbac5c/c64f1e33-0c51-411c-bbbf-0af7b620c655"
-					(reference "R45")
+					(reference "R46")
 					(unit 1)
 				)
@@
 		(in_pos_files yes)
 		(dnp no)
-		(property "Reference" "R36"
+		(property "Reference" "R37"
 			(at 77.47 78.74 90)
 			(show_name no)
@@
 			(project "PS-HVCarrier"
 				(path "/2365a867-6254-4a7c-9718-f325e0bbac5c/c64f1e33-0c51-411c-bbbf-0af7b620c655"
-					(reference "R36")
+					(reference "R37")
 					(unit 1)
 				)
@@
 		(dnp no)
 		(fields_autoplaced yes)
-		(property "Reference" "R47"
+		(property "Reference" "R48"
 			(at 226.06 113.0299 0)
 			(show_name no)
@@
 			(project "PS-HVCarrier"
 				(path "/2365a867-6254-4a7c-9718-f325e0bbac5c/c64f1e33-0c51-411c-bbbf-0af7b620c655"
-					(reference "R47")
+					(reference "R48")
 					(unit 1)
 				)
@@
 		(in_pos_files yes)
 		(dnp no)
-		(property "Reference" "R40"
+		(property "Reference" "R41"
 			(at 154.94 46.99 90)
 			(show_name no)
@@
 			(project "PS-HVCarrier"
 				(path "/2365a867-6254-4a7c-9718-f325e0bbac5c/c64f1e33-0c51-411c-bbbf-0af7b620c655"
-					(reference "R40")
+					(reference "R41")
 					(unit 1)
 				)
@@
 		(dnp no)
 		(fields_autoplaced yes)
-		(property "Reference" "R34"
+		(property "Reference" "R35"
 			(at 77.47 26.67 90)
 			(show_name no)
@@
 			(project "PS-HVCarrier"
 				(path "/2365a867-6254-4a7c-9718-f325e0bbac5c/c64f1e33-0c51-411c-bbbf-0af7b620c655"
-					(reference "R34")
+					(reference "R35")
 					(unit 1)
 				)

Commit message: saving
Parts:
- J10: value SSA-2-100A -> Shunt Conn
Changed lines of the file:
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@@
 			)
 		)
-		(property "Value" "SSA-2-100A"
+		(property "Value" "Shunt Conn"
 			(at 141.478 45.72 0)
 			(show_name no)
