File: hardware/HV_Carrier/Current_Sense.kicad_sch (KiCad schematic)
At the start: 46 parts, among them J10 Shunt Conn, J11 SSA-2-100A, J12 Discharge Vin, J13 Charge Vin, J9 LZSR 80-P, U6 TLV9002QDRQ1

Commit message: missing edgecut
Parts:
- TP14: value SHUNT_OUTP -> SHUNT_UREF
Changed lines of the file:
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@@
 			)
 		)
-		(property "Value" "SHUNT_OUTP"
+		(property "Value" "SHUNT_UREF"
 			(at 167.894 49.784 0)
 			(show_name no)
