File: hardware/HV_Carrier/Voltage_Sense.kicad_sch (KiCad schematic)
At the start: 15 parts

Commit message: CAN stufff
Parts:
- added TP?: MOTOR+ ADC, TestPoint:TestPoint_THTPad_D3.0mm_Drill1.5mm, symbol Connector:TestPoint
- added TP?: HV+ ADC, TestPoint:TestPoint_THTPad_D3.0mm_Drill1.5mm, symbol Connector:TestPoint
- added TP?: MOTOR- ADC, TestPoint:TestPoint_THTPad_D3.0mm_Drill1.5mm, symbol Connector:TestPoint
- added TP?: HV- ADC, TestPoint:TestPoint_THTPad_D3.0mm_Drill1.5mm, symbol Connector:TestPoint
Connections:
- net HV+_ADC: now also TP?.1
- net HV-_ADC: now also TP?.1
- net MOTOR+_ADC: now also TP?.1
- net MOTOR-_ADC: now also TP?.1

Commit message: saving
Parts:
- added TP27: Motor- IN, TestPoint:TestPoint_THTPad_D3.0mm_Drill1.5mm, symbol Connector:TestPoint
- TP26: value MOTOR+ DIAG -> Motor+ DIAG
- TP37: renamed from TP?; value MOTOR+ ADC -> Motor+ ADC
- TP38: renamed from TP?; value MOTOR- ADC -> Motor- ADC
- gave numbers to parts that had none: 2
- renumbered TP27 to TP28, TP28 to TP29, TP29 to TP30, TP30 to TP31, TP31 to TP32, TP32 to TP33, TP33 to TP34
Connections:
- net Motor-: now also TP27.1
Changed lines of the file:
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@@
+	)
+	(junction
+		(at 107.95 105.41)
+		(diameter 0)
+		(color 0 0 0 0)
 	)
 	(junction
@@
 	(wire
 		(pts
-			(xy 105.41 105.41) (xy 111.76 105.41)
+			(xy 105.41 105.41) (xy 107.95 105.41)
+		)
+		(stroke
+			(width 0)
+			(type default)
+		)
+	)
+	(wire
+		(pts
+			(xy 107.95 105.41) (xy 111.76 105.41)
 		)
 		(stroke
@@
 		(in_pos_files yes)
 		(dnp no)
-		(property "Reference" "TP?"
+		(property "Reference" "TP37"
 			(at 224.79 102.1079 0)
 			(hide yes)
@@
 			)
 		)
-		(property "Value" "MOTOR+ ADC"
+		(property "Value" "Motor+ ADC"
 			(at 238.506 100.584 0)
 			(show_name no)
@@
 			(project "PS-HVCarrier"
 				(path "/2365a867-6254-4a7c-9718-f325e0bbac5c/83ab5b0b-4732-42c0-82fe-e74f4113c82a"
-					(reference "TP?")
+					(reference "TP37")
 					(unit 1)
 				)
@@
 		(in_pos_files yes)
 		(dnp no)
-		(property "Reference" "TP32"
+		(property "Reference" "TP33"
 			(at 151.13 51.3079 0)
 			(hide yes)
@@
 			(project "PS-HVCarrier"
 				(path "/2365a867-6254-4a7c-9718-f325e0bbac5c/83ab5b0b-4732-42c0-82fe-e74f4113c82a"
-					(reference "TP32")
+					(reference "TP33")
 					(unit 1)
 				)
@@
 		(in_pos_files yes)
 		(dnp no)
-		(property "Reference" "TP31"
+		(property "Reference" "TP32"
 			(at 148.59 102.1079 0)
 			(hide yes)
@@
 			(project "PS-HVCarrier"
 				(path "/2365a867-6254-4a7c-9718-f325e0bbac5c/83ab5b0b-4732-42c0-82fe-e74f4113c82a"
-					(reference "TP31")
+					(reference "TP32")
 					(unit 1)
 				)
@@
 		(in_pos_files yes)
 		(dnp no)
-		(property "Reference" "TP33"
+		(property "Reference" "TP34"
 			(at 151.13 91.9479 0)
 			(hide yes)
@@
 			(project "PS-HVCarrier"
 				(path "/2365a867-6254-4a7c-9718-f325e0bbac5c/83ab5b0b-4732-42c0-82fe-e74f4113c82a"
-					(reference "TP33")
+					(reference "TP34")
 					(unit 1)
 				)
@@
 			)
 		)
-		(property "Value" "MOTOR+ DIAG"
+		(property "Value" "Motor+ DIAG"
 			(at 89.408 90.932 0)
 			(show_name no)
@@
 		(in_pos_files yes)
 		(dnp no)
-		(property "Reference" "TP29"
+		(property "Reference" "TP30"
 			(at 148.59 61.4679 0)
 			(hide yes)
@@
 			(project "PS-HVCarrier"
 				(path "/2365a867-6254-4a7c-9718-f325e0bbac5c/83ab5b0b-4732-42c0-82fe-e74f4113c82a"
-					(reference "TP29")
+					(reference "TP30")
 					(unit 1)
 				)
@@
 		(in_pos_files yes)
 		(dnp no)
-		(property "Reference" "TP?"
+		(property "Reference" "TP36"
 			(at 223.52 44.9579 0)
 			(hide yes)
@@
 			(project "PS-HVCarrier"
 				(path "/2365a867-6254-4a7c-9718-f325e0bbac5c/83ab5b0b-4732-42c0-82fe-e74f4113c82a"
-					(reference "TP?")
+					(reference "TP36")
 					(unit 1)
 				)
@@
 		(in_pos_files yes)
 		(dnp no)
-		(property "Reference" "TP27"
+		(property "Reference" "TP28"
 			(at 107.95 60.1979 0)
 			(hide yes)
@@
 			(project "PS-HVCarrier"
 				(path "/2365a867-6254-4a7c-9718-f325e0bbac5c/83ab5b0b-4732-42c0-82fe-e74f4113c82a"
-					(reference "TP27")
+					(reference "TP28")
 					(unit 1)
 				)
@@
 		(in_pos_files yes)
 		(dnp no)
-		(property "Reference" "TP?"
+		(property "Reference" "TP38"
 			(at 224.79 114.8079 0)
 			(hide yes)
@@
 			)
 		)
-		(property "Value" "MOTOR- ADC"
+		(property "Value" "Motor- ADC"
 			(at 238.506 113.284 0)
 			(show_name no)
@@
 			(project "PS-HVCarrier"
 				(path "/2365a867-6254-4a7c-9718-f325e0bbac5c/83ab5b0b-4732-42c0-82fe-e74f4113c82a"
-					(reference "TP?")
+					(reference "TP38")
+					(unit 1)
+				)
+			)
+		)
+	)
+	(symbol
+		(lib_id "Connector:TestPoint")
+		(at 107.95 105.41 0)
+		(mirror y)
+		(unit 1)
+		(body_style 1)
+		(exclude_from_sim no)
+		(in_bom yes)
+		(on_board yes)
+		(in_pos_files yes)
+		(dnp no)
+		(property "Reference" "TP27"
+			(at 105.41 100.8379 0)
+			(hide yes)
+			(show_name no)
+			(do_not_autoplace no)
+			(effects
+				(font
+					(size 1.27 1.27)
+				)
+				(justify left)
+			)
+		)
+		(property "Value" "Motor- IN"
+			(at 106.426 102.616 0)
+			(show_name no)
+			(do_not_autoplace no)
+			(effects
+				(font
+					(size 1.27 1.27)
+				)
+				(justify left)
+			)
+		)
+		(property "Footprint" "TestPoint:TestPoint_THTPad_D3.0mm_Drill1.5mm"
+			(at 102.87 105.41 0)
+			(hide yes)
+			(show_name no)
+			(do_not_autoplace no)
+			(effects
+				(font
+					(size 1.27 1.27)
+				)
+			)
+		)
+		(property "Datasheet" ""
+			(at 102.87 105.41 0)
+			(hide yes)
+			(show_name no)
+			(do_not_autoplace no)
+			(effects
+				(font
+					(size 1.27 1.27)
+				)
+			)
+		)
+		(property "Description" "test point"
+			(at 107.95 105.41 0)
+			(hide yes)
+			(show_name no)
+			(do_not_autoplace no)
+			(effects
+				(font
+					(size 1.27 1.27)
+				)
+			)
+		)
+		(pin "1"
+		)
+		(instances
+			(project "PS-HVCarrier"
+				(path "/2365a867-6254-4a7c-9718-f325e0bbac5c/83ab5b0b-4732-42c0-82fe-e74f4113c82a"
+					(reference "TP27")
 					(unit 1)
 				)
@@
 		(in_pos_files yes)
 		(dnp no)
-		(property "Reference" "TP28"
+		(property "Reference" "TP29"
 			(at 148.59 56.3879 0)
 			(hide yes)
@@
 			(project "PS-HVCarrier"
 				(path "/2365a867-6254-4a7c-9718-f325e0bbac5c/83ab5b0b-4732-42c0-82fe-e74f4113c82a"
-					(reference "TP28")
+					(reference "TP29")
 					(unit 1)
 				)
@@
 		(in_pos_files yes)
 		(dnp no)
-		(property "Reference" "TP30"
+		(property "Reference" "TP31"
 			(at 148.59 97.0279 0)
 			(hide yes)
@@
 			(project "PS-HVCarrier"
 				(path "/2365a867-6254-4a7c-9718-f325e0bbac5c/83ab5b0b-4732-42c0-82fe-e74f4113c82a"
-					(reference "TP30")
+					(reference "TP31")
 					(unit 1)
 				)
@@
 		(in_pos_files yes)
 		(dnp no)
-		(property "Reference" "TP?"
+		(property "Reference" "TP35"
 			(at 223.4297 57.6579 0)
 			(hide yes)
@@
 			(project "PS-HVCarrier"
 				(path "/2365a867-6254-4a7c-9718-f325e0bbac5c/83ab5b0b-4732-42c0-82fe-e74f4113c82a"
-					(reference "TP?")
+					(reference "TP35")
 					(unit 1)
 				)
