File: hardware/HV_Carrier/USB-C Connector.kicad_sch (KiCad schematic)
At the start: 6 parts, among them J6 USB_C_Receptacle_USB2.0_16P

Commit message: saving
Connections:
- net USB_DM: no longer J6.A7 (D-), J6.B7 (D-)
- net USB_DP: no longer J6.A6 (D+), J6.B6 (D+)
- new net USB_D+: J6.A6 (D+), J6.B6 (D+)
- new net USB_D-: J6.A7 (D-), J6.B7 (D-)
Changed lines of the file:
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@@
 		)
 	)
-	(hierarchical_label "USB_DP"
+	(hierarchical_label "USB_D+"
 		(shape bidirectional)
 		(at 55.88 49.53 0)
@@
 		)
 	)
-	(hierarchical_label "USB_DM"
+	(hierarchical_label "USB_D-"
 		(shape bidirectional)
 		(at 55.88 44.45 0)

Commit message: ready for review
Connections:
- net USB_DM is gone; now on net USB_D-: D9.2 (D-)
- net USB_DP is gone; now on net USB_D+: D9.1 (D+)
Changed lines of the file:
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@@
 		)
 	)
-	(hierarchical_label "USB_DP"
+	(hierarchical_label "USB_D+"
 		(shape bidirectional)
 		(at 68.58 78.74 180)
@@
 		)
 	)
-	(hierarchical_label "USB_DM"
+	(hierarchical_label "USB_D-"
 		(shape bidirectional)
 		(at 68.58 81.28 180)
