File: hardware/HV_Carrier/KiCAD-Sharepoint/LHRS_Design_Blocks.kicad_blocks/12VBuck.kicad_block/12VBuck.kicad_sch (KiCad schematic)
At the start: 12 parts, among them U1 LMR51635XDDCR

Commit message: saving
Parts:
- removed C4: 47u, Capacitor_SMD:C_1210_3225Metric_Pad1.33x2.70mm_HandSolder, symbol Device:C_Small
- added C4, C5: 22u, Capacitor_SMD:C_1210_3225Metric_Pad1.33x2.70mm_HandSolder, symbol Device:C
- added C6: 3.3u, Capacitor_SMD:C_0805_2012Metric_Pad1.18x1.45mm_HandSolder, symbol Device:C
- C1: LCSC P/N (none) -> C6962403; P/N MSASL168SB5475KTNA01 -> 08055D475KAT4A
- C2: renamed from C5; footprint Capacitor_SMD:C_0805_2012Metric_Pad1.18x1.45mm_HandSolder -> Capacitor_SMD:C_0603_1608Metric_Pad1.08x0.95mm_HandSolder; LCSC P/N (none) -> C6666325
- C3: renamed from C2; LCSC P/N (none) -> C6666325
- L1: footprint LHRS_Passives:SRN8040-150M -> LHRS_Passives:74439369082
- R1: LCSC P/N (none) -> C25803; P/N AE1206BR-07100KL -> CRCW0603100KFKEE
- R2: LCSC P/N (none) -> C844132; P/N ERA-2ARB1912X -> CRCW060319K1FKEAHP
- renumbered TP9 to TP1, TP10 to TP2, TP11 to TP3, TP12 to TP4
Connections:
- net GND: now also C4.2, C5.2, C6.2
- net V_out_5V: now also C4.1, C5.1, C6.1
