File: hardware/Hall_Interface Board/Hall Interface.kicad_pcb (KiCad board)
At the start: 2 copper layers, 73.9 x 27.1 mm, 2 parts, among them J1 Breakout Connector, U1 LZSR_80-P

Commit message: new gebers
Parts:
- added G***: LHRs_LOGO, LHRS_Logos:LHRs_LOGO, F.Cu at (80.1, 75.8)
- added G***: LOGO, LOGO, B.Cu at (131.2, 64.7)
- added G***: LOGO, LOGO, B.Cu at (107.1, 66.3)
- added G***: LOGO, LOGO, B.Cu at (83.1, 65.4)
Other:
- board text added: "9/11/2026"
- board text added: "HV Carrier"
- board text added: "Shuopu Wang"
